Commit message: Add base_footprint

File: src/tracked_robot_description/urdf/tracked_robot_core.urdf.xacro (robot description, xacro)
@@ -29,4 +29,11 @@
     <xacro:property name="sprocket_radius" value="0.06"/>
     <xacro:macro name="robot" params="diff_drive_emulation mimic_enable:=true path_meshes:=package://tracked_robot_description/meshes">
+<link name="base_footprint"/>
+  <!-- The base footprint of the robot is located underneath the chassis -->
+  <joint name="base_joint" type="fixed">
+    <parent link="base_footprint"/>
+    <child link="base_link" />
+    <origin xyz="0.0 0.0 0.1" rpy="0 0 0"/>
+  </joint>
     <link name="base_link">
         <inertial>

File: src/tracked_robot_gazebo/urdf/diff_drive.gazebo.xacro (robot description, xacro)
@@ -20,7 +20,7 @@
             <wheel_diameter>${wheel_radius * 2}</wheel_diameter>
             <!-- Wheel acceleration, in rad/s^2, defaults to 0.0 rad/s^2 -->
-            <wheel_acceleration>0.0</wheel_acceleration>
+            <wheel_acceleration>0.2</wheel_acceleration>
             <!-- Maximum torque which the wheels can produce, in Nm, defaults to 5 Nm -->
-            <max_wheel_torque>15</max_wheel_torque>
+            <max_wheel_torque>5</max_wheel_torque>
             <!-- Odometry frame, defaults to `odom` -->
             <odometry_frame>odom</odometry_frame>

File: src/tracked_robot_gazebo/urdf/tracked_robot.gazebo.xacro (robot description, xacro)
@@ -12,7 +12,7 @@
     <xacro:robot diff_drive_emulation="true" mimic_enable="true" path_meshes="file://$(find tracked_robot_description)/meshes"/>
     <!-- tracked_robot differential drive controller -->
-    <xacro:track_drive parent="base_link"
+    <xacro:track_drive parent="base_footprint"
                        robot_name="$(arg robot_name)"
-                       update_rate="100.0"
+                       update_rate="10.0"
                        wheel_radius="0.06"
                        wheel_separation="0.4"
@@ -20,7 +20,7 @@
     <xacro:track_hand />
     <xacro:track_camera parent="camera_link"
-                        update_rate="100.0" />
+                        update_rate="30.0" />
     <xacro:track_lidar parent="lidar_link"
-                        update_rate="10.0" />
+                        update_rate="30.0" />
     <xacro:track_imu parent="imu_link" />
 </robot>

Commit message: Trying to fix odometry

File: src/tracked_robot_description/urdf/tracked_robot_core.urdf.xacro (robot description, xacro)
@@ -27,5 +27,5 @@
     </material>
     <xacro:property name="M_PI" value="3.14159"/>
-    <xacro:property name="sprocket_radius" value="0.06"/>
+    <xacro:property name="sprocket_radius" value="0.069"/>
     <xacro:macro name="robot" params="diff_drive_emulation mimic_enable:=true path_meshes:=package://tracked_robot_description/meshes">
 <link name="base_footprint"/>

File: src/tracked_robot_gazebo/urdf/imu.gazebo.xacro (robot description, xacro)
@@ -9,11 +9,61 @@
           <remapping>~/out:=data</remapping>
         </ros>
-        <initial_orientation_as_reference>false</initial_orientation_as_reference>
-        <bodyName>imu_link</bodyName>
-        <updateRateHZ>10.0</updateRateHZ>
-        <gaussianNoise>0.0</gaussianNoise>
-        <xyzOffset>0 0 0</xyzOffset>
-        <rpyOffset>0 0 0</rpyOffset>
-        <frameName>imu_link</frameName>
+         <always_on>true</always_on>
+      <update_rate>100</update_rate>
+      <visualize>true</visualize>
+      <imu>
+        <angular_velocity>
+          <x>
+            <noise type="gaussian">
+              <mean>0.0</mean>
+              <stddev>2e-4</stddev>
+              <bias_mean>0.0000075</bias_mean>
+              <bias_stddev>0.0000008</bias_stddev>
+            </noise>
+          </x>
+          <y>
+            <noise type="gaussian">
+              <mean>0.0</mean>
+              <stddev>2e-4</stddev>
+              <bias_mean>0.0000075</bias_mean>
+              <bias_stddev>0.0000008</bias_stddev>
+            </noise>
+          </y>
+          <z>
+            <noise type="gaussian">
+              <mean>0.0</mean>
+              <stddev>2e-4</stddev>
+              <bias_mean>0.0000075</bias_mean>
+              <bias_stddev>0.0000008</bias_stddev>
+            </noise>
+          </z>
+        </angular_velocity>
+        <linear_acceleration>
+          <x>
+            <noise type="gaussian">
+              <mean>0.0</mean>
+              <stddev>1.7e-2</stddev>
+              <bias_mean>0.1</bias_mean>
+              <bias_stddev>0.001</bias_stddev>
+            </noise>
+          </x>
+          <y>
+            <noise type="gaussian">
+              <mean>0.0</mean>
+              <stddev>1.7e-2</stddev>
+              <bias_mean>0.1</bias_mean>
+              <bias_stddev>0.001</bias_stddev>
+            </noise>
+          </y>
+          <z>
+            <noise type="gaussian">
+              <mean>0.0</mean>
+              <stddev>1.7e-2</stddev>
+              <bias_mean>0.1</bias_mean>
+              <bias_stddev>0.001</bias_stddev>
+            </noise>
+          </z>
+        </linear_acceleration>
+      </imu>
       </plugin>
     </sensor>

File: src/tracked_robot_gazebo/urdf/tracked_robot.gazebo.xacro (robot description, xacro)
@@ -14,5 +14,5 @@
                        robot_name="$(arg robot_name)"
                        update_rate="10.0"
-                       wheel_radius="0.06"
+                       wheel_radius="0.069"
                        wheel_separation="0.4"
                        publish_odom_tf="$(arg publish_odom_tf)" />
