Commit message: Office workshop: fix odometry, params, etc.

File: src/tracked_robot_description/urdf/lidar.urdf.xacro (robot description, xacro)
@@ -3,5 +3,5 @@
     <xacro:macro name="lidar"  params="parent">
         <joint name="lidar_sensor_joint" type="fixed">
-            <origin xyz="0.0 0 0.11" rpy="0 0 0" />
+            <origin xyz="0.0 0 0.11" rpy="0 0 3.141" />
             <parent link="${parent}"/>
             <child link="lidar_link"/>
