Commit message: worked variant

File: src/tracked_robot_description/urdf/imu.urdf.xacro (robot description, xacro)
@@ -2,12 +2,14 @@
 <robot name="tracked_robot" xmlns:xacro="http://ros.org/wiki/xacro">
     <xacro:macro name="imu"  params="parent">
-        <joint name="imu_sensor_joint" type="fixed">
-            <origin xyz="0 0 0" rpy="0 0 0"/>
+        <!-- *********************** IMU SETUP *********************************  -->
+        <!-- Each sensor must be attached to a link.                              -->
+        <joint name="imu_joint" type="fixed">
             <parent link="${parent}"/>
             <child link="imu_link"/>
+            <origin xyz="0 0 0" rpy="0 0 0"/>
         </joint>
         <link name="imu_link">
             <collision>
-            <origin xyz="0 0 0" rpy="0 0 0"/>
+            <origin xyz="-0.02 0 0.17" rpy="0 0 0"/>
             <geometry>
             <box size="0.1 0.1 0.1"/>
@@ -27,4 +29,79 @@
             </inertial>
         </link>
+	 <gazebo reference="imu_link">
+	   <sensor name="mpu9250_imu" type="imu">
+		<plugin name="imu_controller" filename="libgazebo_ros_imu_sensor.so">
+		   <ros>
+		     <remapping>~/out:=imu_broadcaster/imu</remapping>
+		   </ros>
+		  <initial_orientation_as_reference>false</initial_orientation_as_reference>
+		</plugin>
+		 <always_on>true</always_on>
+		 <update_rate>100</update_rate>
+		 <visualize>true</visualize>
+		 <imu>
+		   <angular_velocity>
+		     <x>
+		       <noise type="gaussian">
+		         <mean>0.0</mean>
+		         <stddev>2e-4</stddev>
+		       </noise>
+		     </x>
+		     <y>
+		       <noise type="gaussian">
+		         <mean>0.0</mean>
+		         <stddev>2e-4</stddev>
+		       </noise>
+		     </y>
+		     <z>
+		       <noise type="gaussian">
+		         <mean>0.0</mean>
+		         <stddev>2e-4</stddev>
+		       </noise>
+		     </z>
+		   </angular_velocity>
+		   <linear_acceleration>
+		     <x>
+		       <noise type="gaussian">
+		         <mean>0.0</mean>
+		         <stddev>1.7e-2</stddev>
+		       </noise>
+		     </x>
+		     <y>
+		       <noise type="gaussian">
+		         <mean>0.0</mean>
+		         <stddev>1.7e-2</stddev>
+		       </noise>
+		     </y>
+		     <z>
+		       <noise type="gaussian">
+		         <mean>0.0</mean>
+		         <stddev>1.7e-2</stddev>
+		       </noise>
+		     </z>
+		   </linear_acceleration>
+		   <orientation>
+		     <x>
+		       <noise type="gaussian">
+		          <mean>0.0</mean>
+		          <stddev>2e-3</stddev>
+		        </noise>
+		      </x>
+		      <y>
+		        <noise type="gaussian">
+		          <mean>0.0</mean>
+		          <stddev>2e-3</stddev>
+		        </noise>
+		      </y>
+		      <z>
+		        <noise type="gaussian">
+		          <mean>0.0</mean>
+		          <stddev>2e-3</stddev>
+		        </noise>
+		      </z>
+		    </orientation>
+		 </imu>
+	   </sensor>
+	 </gazebo>
     </xacro:macro>
 </robot>

File: src/tracked_robot_description/urdf/lidar.urdf.xacro (robot description, xacro)
@@ -9,5 +9,5 @@
         <link name="lidar_link">
             <collision>
-            <origin xyz="0 0 0" rpy="0 0 0"/>
+            <origin xyz="0.075 0 0.17" rpy="0 0 0"/>
             <geometry>
                 <cylinder radius="0.05" length="0.04"/>
@@ -19,5 +19,5 @@
                 <cylinder radius="0.05" length="0.04"/>
             </geometry>
-            <material name="red"/>
+            <!--material name="red"/-->
             </visual>
             <inertial>

File: src/tracked_robot_description/urdf/track.urdf.xacro (robot description, xacro)
@@ -29,8 +29,8 @@
         <link name="sprocket_${type}">
          <inertial>
-            <mass value="3" />
-            <inertia ixx="1e-3" ixy="0.0" ixz="0.0"
-                 iyy="1e-3" iyz="0.0"
-                 izz="1e-3" />
+            <mass value="1" />
+            <inertia ixx="0.0" ixy="0.0" ixz="0.0"
+                 iyy="0.0" iyz="0.0"
+                 izz="0.0" />
         </inertial>
             <visual>

File: src/tracked_robot_description/urdf/tracked_robot_core.urdf.xacro (robot description, xacro)
@@ -5,4 +5,5 @@
     <xacro:include filename="lidar.urdf.xacro" />
     <xacro:include filename="imu.urdf.xacro" />
+    <xacro:include filename="gps.urdf.xacro" />
     <material name="Black">
         <color rgba="0.1 0.1 0.1 1.0"/>
@@ -50,4 +51,5 @@
     <xacro:lidar parent="base_link" />
     <xacro:imu parent="base_link" />
+    <xacro:gps parent="base_link" />
     </xacro:macro>
 </robot>
