Commit message: next iteration

File: src/tracked_robot_description/urdf/gps.urdf.xacro (robot description, xacro)
@@ -3,9 +3,4 @@
     <xacro:macro name="gps"  params="parent">
         <!-- *********************** GPS SETUP **********************************  -->
-        <joint name="gps_sensor_joint" type="fixed">
-            <parent link="${parent}"/>
-            <child link="gps_link"/>
-            <origin xyz="0.0 0 0.0" rpy="0 0 0"/>
-        </joint>
         <link name="gps_link">
             <collision>
@@ -23,4 +18,9 @@
             </visual>
         </link>
+        <joint name="gps_sensor_joint" type="fixed">
+            <parent link="${parent}"/>
+            <child link="gps_link"/>
+            <origin xyz="0.0 0 0.0" rpy="0 0 0"/>
+        </joint>
     </xacro:macro>
 </robot>

File: src/tracked_robot_description/urdf/imu.urdf.xacro (robot description, xacro)
@@ -4,12 +4,7 @@
         <!-- *********************** IMU SETUP *********************************  -->
         <!-- Each sensor must be attached to a link.                              -->
-        <joint name="imu_joint" type="fixed">
-            <parent link="${parent}"/>
-            <child link="imu_link"/>
-            <origin xyz="0 0 0" rpy="0 0 0"/>
-        </joint>
         <link name="imu_link">
             <collision>
-            <origin xyz="-0.02 0 0.17" rpy="0 0 0"/>
+            <origin xyz="0 0 0" rpy="0 0 0"/>
             <geometry>
             <box size="0.1 0.1 0.1"/>
@@ -29,4 +24,9 @@
             </inertial>
         </link>
+        <joint name="imu_joint" type="fixed">
+            <parent link="base_link"/>
+            <child link="imu_link"/>
+            <origin xyz="-0.02 0 0.17" rpy="0 0 0"/>
+        </joint>
 	 <gazebo reference="imu_link">
 	   <sensor name="mpu9250_imu" type="imu">

File: src/tracked_robot_description/urdf/lidar.urdf.xacro (robot description, xacro)
@@ -2,9 +2,4 @@
 <robot name="tracked_robot" xmlns:xacro="http://ros.org/wiki/xacro">
     <xacro:macro name="lidar"  params="parent">
-        <joint name="lidar_sensor_joint" type="fixed">
-            <origin xyz="0.0 0 0.11" rpy="0 0 3.141" />
-            <parent link="${parent}"/>
-            <child link="lidar_link"/>
-        </joint>
         <link name="lidar_link">
             <collision>
@@ -27,4 +22,9 @@
             </inertial>
         </link>
+        <joint name="lidar_sensor_joint" type="fixed">
+            <origin xyz="0.0 0 0.11" rpy="0 0 3.141" />
+            <parent link="${parent}"/>
+            <child link="lidar_link"/>
+        </joint>
     </xacro:macro>
 </robot>

File: src/tracked_robot_description/urdf/tracked_robot_core.urdf.xacro (robot description, xacro)
@@ -1,4 +1,6 @@
 <?xml version="1.0" ?>
 <robot name="tracked_robot" xmlns:xacro="http://ros.org/wiki/xacro">
+    <xacro:arg name="use_ros2_control" default="true"/>
+    <xacro:arg name="sim_mode" default="false"/>
     <xacro:include filename="track.urdf.xacro" />
     <xacro:include filename="hand.urdf.xacro" />
@@ -28,16 +30,17 @@
     </material>
     <xacro:property name="M_PI" value="3.14159"/>
-    <xacro:property name="sprocket_radius" value="0.069"/>
+    <xacro:property name="sprocket_radius" value="0.02545"/>
+    <!-- 0.02545 0.0529-->
     <xacro:macro name="robot" params="diff_drive_emulation mimic_enable:=true path_meshes:=package://tracked_robot_description/meshes">
-<link name="base_footprint"/>
-  <!-- The base footprint of the robot is located underneath the chassis -->
-  <joint name="base_joint" type="fixed">
-    <parent link="base_footprint"/>
-    <child link="base_link" />
-    <origin xyz="0.0 0.0 0.1" rpy="0 0 0"/>
-  </joint>
+    <link name="base_footprint"/>
+    <!-- The base footprint of the robot is located underneath the chassis -->
+    <joint name="base_joint" type="fixed">
+        <parent link="base_link"/>
+        <child link="base_footprint" />
+        <origin xyz="0.0 0.0 0.07" rpy="0 0 0"/>
+    </joint>
     <link name="base_link">
         <visual>
-            <origin xyz="-0.221 0 -0.05" rpy="1.5707963267949 0 ${M_PI}"/>
+            <origin xyz="-0.221 0 -0.05" rpy="1.5707963267949 0 0"/>
             <geometry>
                 <mesh filename="${path_meshes}/robot_base.stl" scale="1 1 1" />
