Commit message: Add 180 degree lidar

File: src/tracked_robot_description/urdf/hand.urdf.xacro (robot description, xacro)
@@ -4,5 +4,5 @@
     <xacro:macro name="hand"  params="parent">
         <joint name="hand_base_joint" type="fixed">
-            <origin xyz="0.2 0 0.14" rpy="0 0 0" />
+            <origin xyz="0.04 0 0.14" rpy="0 0 0" />
             <parent link="${parent}"/>
             <child link="hand_base"/>
@@ -18,5 +18,5 @@
                 <origin xyz="0 0 0" rpy="0 0 0"/>
                 <geometry>
-                     <cylinder length="0.09" radius="0.06"/>
+                     <cylinder length="0.12" radius="0.06"/>
                 </geometry>
                 <material name="Black" />
@@ -36,7 +36,7 @@
             </inertial>
             <visual>
-                <origin xyz="0.29 0 0" rpy="0 0 0"/>
+                <origin xyz="0.4 0 0" rpy="0 0 0"/>
                 <geometry>
-                     <box size="0.7 0.1 0.01"/>
+                     <box size="0.9 0.1 0.01"/>
                 </geometry>
                 <material name="Black" />

File: src/tracked_robot_description/urdf/lidar.urdf.xacro (robot description, xacro)
@@ -1,15 +1,15 @@
 <?xml version="1.0"?>
 <robot name="tracked_robot" xmlns:xacro="http://ros.org/wiki/xacro">
-    <xacro:macro name="camera"  params="parent">
-        <joint name="camera_sensor_joint" type="fixed">
-            <origin xyz="0.8 0 -0.015" rpy="0 ${M_PI/2} 0"/>
+    <xacro:macro name="lidar"  params="parent">
+        <joint name="lidar_sensor_joint" type="fixed">
+            <origin xyz="0.25 0 0.11" rpy="0 0 0" />
             <parent link="${parent}"/>
-            <child link="camera_link"/>
+            <child link="lidar_link"/>
         </joint>
-        <link name="camera_link">
+        <link name="lidar_link">
             <collision>
             <origin xyz="0 0 0" rpy="0 0 0"/>
             <geometry>
-            <box size="0.1 0.1 0.1"/>
+                <cylinder radius="0.05" length="0.04"/>
             </geometry>
             </collision>
@@ -17,7 +17,7 @@
             <origin xyz="0 0 0" rpy="0 0 0"/>
             <geometry>
-                <box size="0.02 0.02 0.02"/>
+                <cylinder radius="0.05" length="0.04"/>
             </geometry>
-            <material name="Red"/>
+            <material name="red"/>
             </visual>
             <inertial>

File: src/tracked_robot_description/urdf/tracked_robot_core.urdf.xacro (robot description, xacro)
@@ -3,4 +3,5 @@
     <xacro:include filename="track.urdf.xacro" />
     <xacro:include filename="hand.urdf.xacro" />
+    <xacro:include filename="lidar.urdf.xacro" />
     <material name="Black">
         <color rgba="0.1 0.1 0.1 1.0"/>
@@ -44,4 +45,5 @@
     <xacro:track type="right" parent="base_link" radius="${sprocket_radius}" diff_drive_emulation="${diff_drive_emulation}" mimic_enable="${mimic_enable}"/>
     <xacro:hand parent="base_link" />
+    <xacro:lidar parent="base_link" />
     </xacro:macro>
 </robot>

File: src/tracked_robot_gazebo/urdf/tracked_robot.gazebo.xacro (robot description, xacro)
@@ -5,4 +5,5 @@
     <xacro:include filename="$(find tracked_robot_gazebo)/urdf/diff_drive.gazebo.xacro"/>
     <xacro:include filename="$(find tracked_robot_gazebo)/urdf/camera.gazebo.xacro"/>
+    <xacro:include filename="$(find tracked_robot_gazebo)/urdf/lidar.gazebo.xacro"/>
     <xacro:include filename="$(find tracked_robot_gazebo)/urdf/hand.gazebo.xacro"/>
     <xacro:arg name="robot_name" default="tracked_robot" />
@@ -19,3 +20,5 @@
     <xacro:track_camera parent="camera_link"
                         update_rate="100.0" />
+    <xacro:track_lidar parent="lidar_link"
+                        update_rate="10.0" />
 </robot>

Commit message: Fix mine detection and mine avoidance

File: src/tracked_robot_description/urdf/hand.urdf.xacro (robot description, xacro)
@@ -4,5 +4,5 @@
     <xacro:macro name="hand"  params="parent">
         <joint name="hand_base_joint" type="fixed">
-            <origin xyz="0.04 0 0.14" rpy="0 0 0" />
+            <origin xyz="-0.180 0 0.14" rpy="0 0 0" />
             <parent link="${parent}"/>
             <child link="hand_base"/>

File: src/tracked_robot_description/urdf/lidar.urdf.xacro (robot description, xacro)
@@ -3,5 +3,5 @@
     <xacro:macro name="lidar"  params="parent">
         <joint name="lidar_sensor_joint" type="fixed">
-            <origin xyz="0.25 0 0.11" rpy="0 0 0" />
+            <origin xyz="0.0 0 0.11" rpy="0 0 0" />
             <parent link="${parent}"/>
             <child link="lidar_link"/>

File: src/tracked_robot_description/urdf/track.urdf.xacro (robot description, xacro)
@@ -18,5 +18,5 @@
         <xacro:property name="scale" value="0.0046"/>
         <joint name="sprocket_${type}_joint" type="continuous">
-            <origin xyz="0.221 ${orientation * -0.235} -0.05" rpy="${orientation * M_PI/2} 0 0" />
+            <origin xyz="0.0 ${orientation * -0.235} -0.05" rpy="${orientation * M_PI/2} 0 0" />
             <parent link="${parent}"/>
             <child link="sprocket_${type}"/>
@@ -67,5 +67,5 @@
         </gazebo>
         <joint name="wheel_${type}_joint" type="${mimic_type}">
-            <origin xyz="-0.221 ${orientation * -0.235} -0.05" rpy="${orientation * M_PI/2} 0 0" />
+            <origin xyz="-0.442 ${orientation * -0.235} -0.05" rpy="${orientation * M_PI/2} 0 0" />
             <parent link="${parent}"/>
             <child link="wheel_${type}"/>
@@ -112,5 +112,5 @@
         </gazebo>
         <joint name="track_${type}_joint" type="fixed">
-            <origin xyz="0.0 ${orientation * -0.235} -0.05" rpy="${orientation * M_PI/2} 0 0" />
+            <origin xyz="-0.221 ${orientation * -0.235} -0.05" rpy="${orientation * M_PI/2} 0 0" />
             <parent link="${parent}"/>
             <child link="track_${type}"/>

File: src/tracked_robot_description/urdf/tracked_robot_core.urdf.xacro (robot description, xacro)
@@ -38,5 +38,5 @@
     <link name="base_link">
         <visual>
-            <origin xyz="0 0 -0.05" rpy="1.5707963267949 0 ${M_PI}"/>
+            <origin xyz="-0.221 0 -0.05" rpy="1.5707963267949 0 ${M_PI}"/>
             <geometry>
                 <mesh filename="${path_meshes}/robot_base.stl" scale="1 1 1" />

Commit message: Implement backward action to improve mine avoidance

File: src/tracked_robot_description/urdf/hand.urdf.xacro (robot description, xacro)
@@ -19,5 +19,5 @@
                 <origin xyz="0 0 0" rpy="0 0 0"/>
                 <geometry>
-                     <cylinder length="0.12" radius="0.06"/>
+                     <cylinder length="0.18" radius="0.06"/>
                 </geometry>
                 <material name="Black" />
@@ -25,5 +25,5 @@
         </link>
        <joint name="hand_joint" type="fixed">
-            <origin xyz="0 0 0.05" rpy="0 0 0" />
+            <origin xyz="0 0 0.09" rpy="0 0 0" />
             <parent link="hand_base"/>
             <child link="hand"/>
@@ -32,5 +32,5 @@
         <link name="hand">
             <visual>
-                <origin xyz="0.3     0 0" rpy="0 0 0"/>
+                <origin xyz="0.3 0 0" rpy="0 0 0"/>
                 <geometry>
                      <box size="0.7 0.1 0.01"/>

Commit message: Update algorithm to avoid big obstacles on field

File: src/tracked_robot_description/urdf/hand.urdf.xacro (robot description, xacro)
@@ -4,5 +4,5 @@
     <xacro:macro name="hand"  params="parent">
         <joint name="hand_base_joint" type="fixed">
-            <origin xyz="-0.180 0 0.14" rpy="0 0 0" />
+            <origin xyz="0.0 0 0.14" rpy="0 0 0" />
             <parent link="${parent}"/>
             <child link="hand_base"/>

File: src/tracked_robot_description/urdf/lidar.urdf.xacro (robot description, xacro)
@@ -3,5 +3,5 @@
     <xacro:macro name="lidar"  params="parent">
         <joint name="lidar_sensor_joint" type="fixed">
-            <origin xyz="0.0 0 0.11" rpy="0 0 0" />
+            <origin xyz="0.221 0 0.11" rpy="0 0 0" />
             <parent link="${parent}"/>
             <child link="lidar_link"/>

File: src/tracked_robot_description/urdf/track.urdf.xacro (robot description, xacro)
@@ -67,5 +67,5 @@
         </gazebo>
         <joint name="wheel_${type}_joint" type="${mimic_type}">
-            <origin xyz="-0.442 ${orientation * -0.235} -0.05" rpy="${orientation * M_PI/2} 0 0" />
+            <origin xyz="-0.221 ${orientation * -0.235} -0.05" rpy="${orientation * M_PI/2} 0 0" />
             <parent link="${parent}"/>
             <child link="wheel_${type}"/>
@@ -112,5 +112,5 @@
         </gazebo>
         <joint name="track_${type}_joint" type="fixed">
-            <origin xyz="-0.221 ${orientation * -0.235} -0.05" rpy="${orientation * M_PI/2} 0 0" />
+            <origin xyz="0.0 ${orientation * -0.235} -0.05" rpy="${orientation * M_PI/2} 0 0" />
             <parent link="${parent}"/>
             <child link="track_${type}"/>

File: src/tracked_robot_description/urdf/tracked_robot_core.urdf.xacro (robot description, xacro)
@@ -39,5 +39,5 @@
     <link name="base_link">
         <visual>
-            <origin xyz="-0.221 0 -0.05" rpy="1.5707963267949 0 ${M_PI}"/>
+            <origin xyz="0.0 0 -0.05" rpy="1.5707963267949 0 ${M_PI}"/>
             <geometry>
                 <mesh filename="${path_meshes}/robot_base.stl" scale="1 1 1" />
