Commit message: fix robot model and improve field planing

File: src/tracked_robot_description/urdf/hand.urdf.xacro (robot description, xacro)
@@ -2,37 +2,37 @@
 <robot name="tracked_robot" xmlns:xacro="http://ros.org/wiki/xacro">
     <xacro:include filename="camera.urdf.xacro" />
-    <xacro:macro name="hand"  params="parent">
+    <xacro:macro name="hand" params="parent">
         <joint name="hand_base_joint" type="fixed">
             <origin xyz="0.0 0 0.14" rpy="0 0 0" />
-            <parent link="${parent}"/>
-            <child link="hand_base"/>
+            <parent link="${parent}" />
+            <child link="hand_base" />
             <axis xyz="0 0 1" />
         </joint>
         <link name="hand_base">
-        <inertial>
-            <mass value="2" />
-            <inertia ixx="1e-3" ixy="0.0" ixz="0.0"
-                 iyy="1e-3" iyz="0.0"
-                 izz="1e-3" />
-        </inertial>
+            <inertial>
+                <mass value="0.2" />
+                <inertia ixx="1e-3" ixy="0.0" ixz="0.0"
+                    iyy="1e-3" iyz="0.0"
+                    izz="1e-3" />
+            </inertial>
             <visual>
-                <origin xyz="0 0 0" rpy="0 0 0"/>
+                <origin xyz="0 0 0" rpy="0 0 0" />
                 <geometry>
-                     <cylinder length="0.36" radius="0.06"/>
+                    <cylinder length="0.36" radius="0.06" />
                 </geometry>
                 <material name="Black" />
             </visual>
         </link>
-       <joint name="hand_joint" type="fixed">
+        <joint name="hand_joint" type="fixed">
             <origin xyz="0 0 0.18" rpy="0 0 0" />
-            <parent link="hand_base"/>
-            <child link="hand"/>
+            <parent link="hand_base" />
+            <child link="hand" />
             <axis xyz="0 0 1" />
         </joint>
         <link name="hand">
             <visual>
-                <origin xyz="0.3 0 0" rpy="0 0 0"/>
+                <origin xyz="0.3 0 0" rpy="0 0 0" />
                 <geometry>
-                     <box size="0.7 0.1 0.01"/>
+                    <box size="0.7 0.1 0.01" />
                 </geometry>
                 <material name="Black" />

File: src/tracked_robot_description/urdf/track.urdf.xacro (robot description, xacro)
@@ -4,39 +4,39 @@
         <!-- Define orientation -->
         <xacro:if value="${type == 'left'}">
-            <xacro:property name="orientation" value="-1"/>
+            <xacro:property name="orientation" value="-1" />
         </xacro:if>
         <xacro:if value="${type == 'right'}">
-            <xacro:property name="orientation" value="1"/>
+            <xacro:property name="orientation" value="1" />
         </xacro:if>
         <xacro:if value="${mimic_enable}">
-            <xacro:property name="mimic_type" value="continuous"/>
+            <xacro:property name="mimic_type" value="continuous" />
         </xacro:if>
         <xacro:unless value="${mimic_enable}">
-            <xacro:property name="mimic_type" value="fixed"/>
+            <xacro:property name="mimic_type" value="fixed" />
         </xacro:unless>
-        <xacro:property name="radius_wheel" value="${radius}"/>
-        <xacro:property name="scale" value="0.0046"/>
+        <xacro:property name="radius_wheel" value="${radius}" />
+        <xacro:property name="scale" value="0.0046" />
         <joint name="sprocket_${type}_joint" type="continuous">
             <origin xyz="0.0 ${orientation * -0.235} -0.05" rpy="${orientation * M_PI/2} 0 0" />
-            <parent link="${parent}"/>
-            <child link="sprocket_${type}"/>
+            <parent link="${parent}" />
+            <child link="sprocket_${type}" />
             <axis xyz="0 0 ${-1 * orientation}" />
             <!-- Passive wheel rotate automatically according to the status of the active one -->
             <xacro:if value="${mimic_enable}">
-                <mimic joint="wheel_${type}_joint" multiplier="1" offset="0"/>
+                <mimic joint="wheel_${type}_joint" multiplier="1" offset="0" />
             </xacro:if>
         </joint>
         <link name="sprocket_${type}">
-         <inertial>
-            <mass value="3" />
-            <inertia ixx="1e-3" ixy="0.0" ixz="0.0"
-                 iyy="1e-3" iyz="0.0"
-                 izz="1e-3" />
-        </inertial>
-            <visual>
-                <origin xyz="0 0 0" rpy="0 0 0" />
-                <geometry>
-                    <mesh filename="${path_meshes}/sprocket.stl" scale="${scale} ${scale} ${scale}"/>
-                    <cylinder length="0.06" radius="${radius_wheel}"/>
+            <inertial>
+                <mass value="0.1" />
+                <inertia ixx="1e-3" ixy="0.0" ixz="0.0"
+                    iyy="1e-3" iyz="0.0"
+                    izz="1e-3" />
+            </inertial>
+            <visual>
+                <origin xyz="0 0 0" rpy="0 0 0" />
+                <geometry>
+                    <mesh filename="${path_meshes}/sprocket.stl" scale="${scale} ${scale} ${scale}" />
+                    <cylinder length="0.06" radius="${radius_wheel}" />
                 </geometry>
                 <material name="Black" />
@@ -46,5 +46,5 @@
                 <origin xyz="0 0 0" rpy="0 0 0" />
                 <geometry>
-                    <cylinder length="0.06" radius="${radius}"/>
+                    <cylinder length="0.06" radius="${radius}" />
                 </geometry>
                 <material name="Black" />
@@ -53,6 +53,6 @@
         <gazebo reference="sprocket_${type}">
             <material>Gazebo/Blue</material>
-            <kp>10000000</kp>
-            <kd>10000000</kd>
+            <kp>1e15</kp>
+            <kd>1e13</kd>
             <mu1>10000000</mu1>
             <mu2>10000000</mu2>
@@ -68,20 +68,20 @@
         <joint name="wheel_${type}_joint" type="${mimic_type}">
             <origin xyz="-0.221 ${orientation * -0.235} -0.05" rpy="${orientation * M_PI/2} 0 0" />
-            <parent link="${parent}"/>
-            <child link="wheel_${type}"/>
+            <parent link="${parent}" />
+            <child link="wheel_${type}" />
             <axis xyz="0 0 ${-1 * orientation}" />
         </joint>
         <link name="wheel_${type}">
-        <inertial>
-            <mass value="3" />
-            <inertia ixx="1e-3" ixy="0.0" ixz="0.0"
-                 iyy="1e-3" iyz="0.0"
-                 izz="1e-3" />
-        </inertial>
-            <visual>
-                <origin xyz="0 0 0" rpy="0 0 0" />
-                <geometry>
-                    <mesh filename="${path_meshes}/wheel.stl" scale="${scale} ${scale} ${scale}"/>
-                    <cylinder length="0.06" radius="${radius_wheel}"/>
+            <inertial>
+                <mass value="0.1" />
+                <inertia ixx="1e-3" ixy="0.0" ixz="0.0"
+                    iyy="1e-3" iyz="0.0"
+                    izz="1e-3" />
+            </inertial>
+            <visual>
+                <origin xyz="0 0 0" rpy="0 0 0" />
+                <geometry>
+                    <mesh filename="${path_meshes}/wheel.stl" scale="${scale} ${scale} ${scale}" />
+                    <cylinder length="0.06" radius="${radius_wheel}" />
                 </geometry>
                 <material name="Black" />
@@ -91,5 +91,5 @@
                 <origin xyz="0 0 0" rpy="0 0 0" />
                 <geometry>
-                    <cylinder length="0.06" radius="${radius_wheel}"/>
+                    <cylinder length="0.06" radius="${radius_wheel}" />
                 </geometry>
                 <material name="Black" />
@@ -98,6 +98,6 @@
         <gazebo reference="wheel_${type}">
             <material>Gazebo/Red</material>
-            <kp>10000000</kp>
-            <kd>10000000</kd>
+            <kp>1e15</kp>
+            <kd>1e13</kd>
             <mu1>0</mu1>
             <mu2>0</mu2>
@@ -111,21 +111,82 @@
             </visual>
         </gazebo>
-        <joint name="track_${type}_joint" type="fixed">
-            <origin xyz="0.0 ${orientation * -0.235} -0.05" rpy="${orientation * M_PI/2} 0 0" />
-            <parent link="${parent}"/>
-            <child link="track_${type}"/>
+        <joint name="front_wheel_${type}_joint" type="${mimic_type}">
+            <origin xyz="0.221 ${orientation * -0.235} -0.05" rpy="${orientation * M_PI/2} 0 0" />
+            <parent link="${parent}" />
+            <child link="front_wheel_${type}" />
+            <axis xyz="0 0 ${-1 * orientation}" />
+        </joint>
+        <link name="front_wheel_${type}">
+            <inertial>
+                <mass value="0.1" />
+                <inertia ixx="1e-3" ixy="0.0" ixz="0.0"
+                    iyy="1e-3" iyz="0.0"
+                    izz="1e-3" />
+            </inertial>
+            <visual>
+                <origin xyz="0 0 0" rpy="0 0 0" />
+                <geometry>
+                    <mesh filename="${path_meshes}/wheel.stl" scale="${scale} ${scale} ${scale}" />
+                    <cylinder length="0.06" radius="${radius_wheel}" />
+                </geometry>
+                <material name="Black" />
+            </visual>
+            <!-- Collision cylinder -->
+            <collision>
+                <origin xyz="0 0 0" rpy="0 0 0" />
+                <geometry>
+                    <cylinder length="0.06" radius="${radius_wheel}" />
+                </geometry>
+                <material name="Black" />
+            </collision>
+        </link>
+        <gazebo reference="front_wheel_${type}">
+            <material>Gazebo/Red</material>
+            <kp>1e15</kp>
+            <kd>1e13</kd>
+            <mu1>0</mu1>
+            <mu2>0</mu2>
+            <!-- Ignition color reference -->
+            <visual>
+                <material>
+                    <ambient>0.5 0.0 0.0 1.0</ambient>
+                    <diffuse>0.5 0.0 0.0 1.0</diffuse>
+                    <specular>0.5 0.0 0.0 1.0</specular>
+                </material>
+            </visual>
+        </gazebo>
+        <joint name="track_${type}_joint" type="continuous">
+            <origin xyz="0.0 ${orientation * -0.235} -0.05" rpy="0 0 0" />
+            <parent link="${parent}" />
+            <child link="track_${type}" />
         </joint>
         <link name="track_${type}">
-            <visual>
-                <origin xyz="0 0 0" rpy="${M_PI/2} 0 0" />
-                <geometry>
-                    <mesh filename="${path_meshes}/track.stl" scale="${scale} ${scale} ${scale}"/>
-                </geometry>
-                <material name="Black" />
-            </visual>
+            <inertial>
+                <mass value="0.2" />
+                <inertia ixx="1e-3" ixy="0.0" ixz="0.0"
+                    iyy="1e-3" iyz="0.0"
+                    izz="1e-3" />
+            </inertial>
+            <visual>
+                <origin xyz="0 0 0" rpy="0 0 0" />
+                <geometry>
+                    <mesh filename="${path_meshes}/track.stl" scale="${scale} ${scale} ${scale}" />
+                </geometry>
+                <material name="Black" />
+            </visual>
+            <collision>
+                <origin xyz="0 0 0" rpy="0 0 0" />
+                <geometry>
+                    <box size="0.56 0.07 0.12" />
+                </geometry>
+                <material name="Black" />
+            </collision>
         </link>
         <gazebo reference="track_${type}">
             <material>Gazebo/Black</material>
-            <!-- Ignition color reference -->
+            <kp>1e15</kp>
+            <kd>1e13</kd>
+            <mu1>0</mu1>
+            <mu2>0</mu2>
             <visual>
                 <material>

File: src/tracked_robot_description/urdf/tracked_robot_core.urdf.xacro (robot description, xacro)
@@ -1,3 +1,3 @@
-<?xml version="1.0" ?>
+<?xml version="1.0"?>
 <robot name="tracked_robot" xmlns:xacro="http://ros.org/wiki/xacro">
     <xacro:include filename="track.urdf.xacro" />
@@ -7,17 +7,17 @@
     <xacro:include filename="gps.urdf.xacro" />
     <material name="Black">
-        <color rgba="0.1 0.1 0.1 1.0"/>
+        <color rgba="0.1 0.1 0.1 1.0" />
     </material>
     <material name="Green">
-        <color rgba="0.0 0.8 0.0 1.0"/>
+        <color rgba="0.0 0.8 0.0 1.0" />
     </material>
     <material name="aluminum">
-        <color rgba="0.5 0.5 0.5 1.0"/>
+        <color rgba="0.5 0.5 0.5 1.0" />
     </material>
     <material name="DarkGrey">
-        <color rgba="0.3 0.3 0.3 1.0"/>
+        <color rgba="0.3 0.3 0.3 1.0" />
     </material>
     <material name="GunMetalGrey">
-        <color rgba="0.46 0.5 0.56 1.0"/>
+        <color rgba="0.46 0.5 0.56 1.0" />
     </material>
     <material name="Gold">
@@ -25,31 +25,47 @@
     </material>
     <material name="zedm_mat">
-        <color rgba="0 0 0 0.9"/>
+        <color rgba="0 0 0 0.9" />
     </material>
-    <xacro:property name="M_PI" value="3.14159"/>
-    <xacro:property name="sprocket_radius" value="0.069"/>
-    <xacro:macro name="robot" params="diff_drive_emulation mimic_enable:=true path_meshes:=package://tracked_robot_description/meshes">
-<link name="base_footprint"/>
-  <!-- The base footprint of the robot is located underneath the chassis -->
-  <joint name="base_joint" type="fixed">
-    <parent link="base_footprint"/>
-    <child link="base_link" />
-    <origin xyz="0.0 0.0 0.1" rpy="0 0 0"/>
-  </joint>
-    <link name="base_link">
-        <visual>
-            <origin xyz="0.0 0 -0.05" rpy="1.5707963267949 0 ${M_PI}"/>
-            <geometry>
-                <mesh filename="${path_meshes}/robot_base.stl" scale="1 1 1" />
-            </geometry>
-            <material name="Green" />
-        </visual>
-    </link>
-    <xacro:track type="left" parent="base_link" radius="${sprocket_radius}" diff_drive_emulation="${diff_drive_emulation}" mimic_enable="${mimic_enable}"/>
-    <xacro:track type="right" parent="base_link" radius="${sprocket_radius}" diff_drive_emulation="${diff_drive_emulation}" mimic_enable="${mimic_enable}"/>
-    <xacro:hand parent="base_link" />
-    <xacro:lidar parent="base_link" />
-    <xacro:imu parent="base_link" />
-    <xacro:gps parent="base_link" />
+    <xacro:property name="M_PI" value="3.14159" />
+    <xacro:property name="sprocket_radius" value="0.069" />
+    <xacro:macro name="robot"
+        params="diff_drive_emulation mimic_enable:=true path_meshes:=package://tracked_robot_description/meshes">
+        <link name="base_footprint" />
+        <!-- The base footprint of the robot is located underneath the chassis -->
+        <joint name="base_joint" type="fixed">
+            <parent link="base_footprint" />
+            <child link="base_link" />
+            <origin xyz="0.0 0.0 0.1" rpy="0 0 0" />
+        </joint>
+        <link name="base_link">
+            <inertial>
+                <mass value="0.5" />
+                <inertia ixx="1e-3" ixy="0.0" ixz="0.0"
+                    iyy="1e-3" iyz="0.0"
+                    izz="1e-3" />
+            </inertial>
+            <visual>
+                <origin xyz="0.0 0 -0.05" rpy="1.5707963267949 0 ${M_PI}" />
+                <geometry>
+                    <mesh filename="${path_meshes}/robot_base.stl" scale="1 1 1" />
+                </geometry>
+                <material name="Green" />
+            </visual>
+            <collision>
+                <origin xyz="0 0 0" rpy="0 0 0" />
+                <geometry>
+                    <box size="0.6 0.36 0.2" />
+                </geometry>
+                <material name="Black" />
+            </collision>
+        </link>
+        <xacro:track type="left" parent="base_link" radius="${sprocket_radius}"
+            diff_drive_emulation="${diff_drive_emulation}" mimic_enable="${mimic_enable}" />
+        <xacro:track type="right" parent="base_link" radius="${sprocket_radius}"
+            diff_drive_emulation="${diff_drive_emulation}" mimic_enable="${mimic_enable}" />
+        <xacro:hand parent="base_link" />
+        <xacro:lidar parent="base_link" />
+        <xacro:imu parent="base_link" />
+        <xacro:gps parent="base_link" />
     </xacro:macro>
 </robot>

File: src/tracked_robot_gazebo/urdf/diff_drive.gazebo.xacro (robot description, xacro)
@@ -1,51 +1,58 @@
 <?xml version="1.0"?>
 <robot name="tracked_robot" xmlns:xacro="http://ros.org/wiki/xacro">
-    <!--Reference http://gazebosim.org/tutorials?tut=ros_gzplugins#DifferentialDrive -->
-    <xacro:macro name="track_drive" params="parent robot_name update_rate wheel_radius wheel_separation publish_odom_tf">
+    <!--Reference
+    http://gazebosim.org/tutorials?tut=ros_gzplugins#DifferentialDrive -->
+    <xacro:macro name="track_drive"
+        params="parent robot_name update_rate wheel_radius wheel_separation publish_odom_tf">
         <gazebo>
             <plugin filename="libgazebo_ros_diff_drive.so" name="skid_steer_drive_controller">
-            <!-- Plugin update rate in Hz -->
-            <update_rate>${update_rate}</update_rate>
-            <num_wheel_pairs>2</num_wheel_pairs>
-            <!-- Name of left joint, defaults to `left_joint` -->
-            <left_joint>sprocket_left_joint</left_joint>
-            <!-- Name of right joint, defaults to `right_joint` -->
-            <right_joint>sprocket_right_joint</right_joint>
-            <left_joint>wheel_left_joint</left_joint>
-            <!-- Name of right joint, defaults to `right_joint` -->
-            <right_joint>wheel_right_joint</right_joint>
-            <!-- The distance from the center of one wheel to the other, in meters, defaults to 0.34 m -->
-            <wheel_separation>${wheel_separation}</wheel_separation>
-            <!-- Diameter of the wheels, in meters, defaults to 0.15 m -->
-            <wheel_diameter>${wheel_radius * 2}</wheel_diameter>
-            <!-- Wheel acceleration, in rad/s^2, defaults to 0.0 rad/s^2 -->
-            <wheel_acceleration>0.2</wheel_acceleration>
-            <!-- Maximum torque which the wheels can produce, in Nm, defaults to 5 Nm -->
-            <max_wheel_torque>5</max_wheel_torque>
-            <!-- Odometry frame, defaults to `odom` -->
-            <odometry_frame>odom</odometry_frame>
-            <!-- Robot frame to calculate odometry from, defaults to `base_footprint` -->
-            <robot_base_frame>${parent}</robot_base_frame>
-            <!-- Set to true to publish transforms for the odometry, defaults to true -->
-            <publish_odom>true</publish_odom>
-            <publish_odom_tf>${publish_odom_tf}</publish_odom_tf>
-            <!-- Set to true to publish transforms for the wheel links, defaults to false -->
-            <publish_wheel_tf>false</publish_wheel_tf>
-            <!-- Odometry source, 0 for ENCODER, 1 for WORLD, defaults to WORLD -->
-            <odometry_source>1</odometry_source>
-            <!-- Set to true to publish sensor_msgs/JointState on /joint_states for the wheel joints, defaults to false -->
-            <publis_wheel_joint_state>false</publis_wheel_joint_state>
+                <!-- Plugin update rate in Hz -->
+                <update_rate>${update_rate}</update_rate>
+                <num_wheel_pairs>3</num_wheel_pairs>
+                <!-- Name of left joint, defaults to `left_joint` -->
+                <left_joint>sprocket_left_joint</left_joint>
+                <!-- Name of right joint, defaults to `right_joint` -->
+                <right_joint>sprocket_right_joint</right_joint>
+                <left_joint>wheel_left_joint</left_joint>
+                <!-- Name of right joint, defaults to `right_joint` -->
+                <right_joint>wheel_right_joint</right_joint>
+                <left_joint>front_wheel_left_joint</left_joint>
+                <!-- Name of right joint, defaults to `right_joint` -->
+                <right_joint>front_wheel_right_joint</right_joint>
+                <!-- The distance from the center of one wheel to the other, in meters, defaults to
+                0.34 m -->
+                <wheel_separation>${wheel_separation}</wheel_separation>
+                <!-- Diameter of the wheels, in meters, defaults to 0.15 m -->
+                <wheel_diameter>${wheel_radius * 2}</wheel_diameter>
+                <!-- Wheel acceleration, in rad/s^2, defaults to 0.0 rad/s^2 -->
+                <wheel_acceleration>0.2</wheel_acceleration>
+                <!-- Maximum torque which the wheels can produce, in Nm, defaults to 5 Nm -->
+                <max_wheel_torque>5</max_wheel_torque>
+                <!-- Odometry frame, defaults to `odom` -->
+                <odometry_frame>odom</odometry_frame>
+                <!-- Robot frame to calculate odometry from, defaults to `base_footprint` -->
+                <robot_base_frame>${parent}</robot_base_frame>
+                <!-- Set to true to publish transforms for the odometry, defaults to true -->
+                <publish_odom>true</publish_odom>
+                <publish_odom_tf>${publish_odom_tf}</publish_odom_tf>
+                <!-- Set to true to publish transforms for the wheel links, defaults to false -->
+                <publish_wheel_tf>false</publish_wheel_tf>
+                <!-- Odometry source, 0 for ENCODER, 1 for WORLD, defaults to WORLD -->
+                <odometry_source>1</odometry_source>
+                <!-- Set to true to publish sensor_msgs/JointState on /joint_states for the wheel
+                joints, defaults to false -->
+                <publis_wheel_joint_state>false</publis_wheel_joint_state>
             </plugin>
             <plugin name="basic_mobile_bot_joint_state"
-            filename="libgazebo_ros_joint_state_publisher.so">
-            <ros>
-                <remapping>~/out:=joint_states</remapping>
-            </ros>
-            <update_rate>${update_rate}</update_rate>
-            <joint_name>sprocket_left_joint</joint_name>
-            <joint_name>sprocket_right_joint</joint_name>
-            <joint_name>wheel_left_joint</joint_name>
-            <joint_name>wheel_right_joint</joint_name>
-        </plugin>
+                filename="libgazebo_ros_joint_state_publisher.so">
+                <ros>
+                    <remapping>~/out:=joint_states</remapping>
+                </ros>
+                <update_rate>${update_rate}</update_rate>
+                <joint_name>sprocket_left_joint</joint_name>
+                <joint_name>sprocket_right_joint</joint_name>
+                <joint_name>wheel_left_joint</joint_name>
+                <joint_name>wheel_right_joint</joint_name>
+            </plugin>
         </gazebo>
     </xacro:macro>
