Commit message: Fix robot wheels

File: src/tracked_robot_description/urdf/track.urdf.xacro (robot description, xacro)
@@ -33,4 +33,5 @@
                 <geometry>
                     <mesh filename="${path_meshes}/sprocket.stl" scale="${scale} ${scale} ${scale}"/>
+                    <cylinder length="0.06" radius="${radius_wheel}"/>
                 </geometry>
                 <material name="Black" />
@@ -40,5 +41,5 @@
                 <origin xyz="0 0 0" rpy="0 0 0" />
                 <geometry>
-                    <cylinder length="0.015" radius="${radius}"/>
+                    <cylinder length="0.06" radius="${radius}"/>
                 </geometry>
                 <material name="Black" />
@@ -80,4 +81,5 @@
                 <geometry>
                     <mesh filename="${path_meshes}/wheel.stl" scale="${scale} ${scale} ${scale}"/>
+                    <cylinder length="0.06" radius="${radius_wheel}"/>
                 </geometry>
                 <material name="Black" />
@@ -87,5 +89,5 @@
                 <origin xyz="0 0 0" rpy="0 0 0" />
                 <geometry>
-                    <cylinder length="0.015" radius="${radius_wheel}"/>
+                    <cylinder length="0.06" radius="${radius_wheel}"/>
                 </geometry>
                 <material name="Black" />
@@ -107,53 +109,4 @@
             </visual>
         </gazebo>
-        <xacro:if value="${diff_drive_emulation}">
-            <joint name="front_wheel_${type}_joint" type="${mimic_type}">
-                <origin xyz="-0.221 ${orientation * -0.235} -0.05" rpy="${orientation * M_PI/2} 0 0" />
-                <parent link="${parent}"/>
-                <child link="front_wheel_${type}"/>
-                <axis xyz="0 0 ${-1 * orientation}" />
-                <!-- Passive sprocket rotate automatically according to the status of the active one -->
-                <xacro:if value="${mimic_enable}">
-                    <mimic joint="sprocket_${type}_joint" multiplier="1" offset="0"/>
-                </xacro:if>
-            </joint>
-            <link name="front_wheel_${type}">
-                <inertial>
-                    <mass value="0.01"/>
-                    <origin rpy=" 0 0 0" xyz="0 0 0"/>
-                    <inertia ixx="1.6666666666666668e-07" ixy="0" ixz="0" iyy="1.6666666666666668e-07" iyz="0" izz="1.6666666666666668e-07"/>
-                </inertial>
-                <visual>
-                    <origin xyz="0 0 0" rpy="0 0 0" />
-                    <geometry>
-                        <mesh filename="${path_meshes}/wheel.stl" scale="${scale} ${scale} ${scale}"/>
-                    </geometry>
-                    <material name="Black" />
-                </visual>
-                <!-- Collision cylinder -->
-                <collision>
-                    <origin xyz="0 0 0" rpy="0 0 0" />
-                    <geometry>
-                        <cylinder length="0.015" radius="${radius_wheel}"/>
-                    </geometry>
-                    <material name="Black" />
-                </collision>
-            </link>
-            <gazebo reference="front_wheel_${type}">
-                <kp>10000000</kp>
-                <kd>10000000</kd>
-                <mu1>0</mu1>
-                <mu2>0</mu2>
-                <material>Gazebo/Green</material>
-                <!-- Ignition color reference -->
-                <visual>
-                    <material>
-                        <ambient>0.0 0.5 0.0 1.0</ambient>
-                        <diffuse>0.0 0.5 0.0 1.0</diffuse>
-                        <specular>0.0 0.5 0.0 1.0</specular>
-                    </material>
-                </visual>
-            </gazebo>
-        </xacro:if>
         <joint name="track_${type}_joint" type="fixed">
             <origin xyz="0.0 ${orientation * -0.235} -0.05" rpy="${orientation * M_PI/2} 0 0" />

File: src/tracked_robot_description/urdf/tracked_robot_core.urdf.xacro (robot description, xacro)
@@ -24,5 +24,5 @@
     </material>
     <xacro:property name="M_PI" value="3.14159"/>
-    <xacro:property name="sprocket_radius" value="0.150"/>
+    <xacro:property name="sprocket_radius" value="0.06"/>
     <xacro:macro name="robot" params="diff_drive_emulation mimic_enable:=true path_meshes:=package://tracked_robot_description/meshes">
     <link name="base_link">

File: src/tracked_robot_gazebo/urdf/diff_drive.gazebo.xacro (robot description, xacro)
@@ -5,18 +5,10 @@
         <gazebo>
             <plugin filename="libgazebo_ros_diff_drive.so" name="skid_steer_drive_controller">
-            <ros>
-                <namespace>${robot_name}</namespace>
-                <argument>--ros-args --remap /cmd_vel:=cmd_vel</argument>
-                <argument>--ros-args --remap /odom:=odom</argument>
-            </ros>
             <!-- Plugin update rate in Hz -->
             <update_rate>${update_rate}</update_rate>
-            <num_wheel_pairs>2</num_wheel_pairs>
             <!-- Name of left joint, defaults to `left_joint` -->
             <left_joint>sprocket_left_joint</left_joint>
-            <left_joint>wheel_left_joint</left_joint>
             <!-- Name of right joint, defaults to `right_joint` -->
             <right_joint>sprocket_right_joint</right_joint>
-            <right_joint>wheel_right_joint</right_joint>
             <!-- The distance from the center of one wheel to the other, in meters, defaults to 0.34 m -->
             <wheel_separation>${wheel_separation}</wheel_separation>

File: src/tracked_robot_gazebo/urdf/tracked_robot.gazebo.xacro (robot description, xacro)
@@ -5,13 +5,11 @@
     <xacro:include filename="$(find tracked_robot_gazebo)/urdf/diff_drive.gazebo.xacro"/>
     <xacro:arg name="robot_name" default="tracked_robot" />
-    <!-- camera definitions -->
-    <xacro:arg name="publish_pointcloud"  default="false"/>
-    <xacro:arg name="publish_odom_tf"  default="false"/>
-    <xacro:robot diff_drive_emulation="true" path_meshes="file://$(find tracked_robot_description)/meshes"/>
+    <xacro:arg name="publish_odom_tf"  default="true"/>
+    <xacro:robot diff_drive_emulation="true" mimic_enable="false" path_meshes="file://$(find tracked_robot_description)/meshes"/>
     <!-- tracked_robot differential drive controller -->
     <xacro:track_drive parent="base_link"
                        robot_name="$(arg robot_name)"
                        update_rate="100.0"
-                       wheel_radius="0.150"
+                       wheel_radius="0.06"
                        wheel_separation="0.4"
                        publish_odom_tf="$(arg publish_odom_tf)" />

Commit message: Fix wheel rotation issue

File: src/tracked_robot_description/urdf/track.urdf.xacro (robot description, xacro)
@@ -22,4 +22,8 @@
             <child link="sprocket_${type}"/>
             <axis xyz="0 0 ${-1 * orientation}" />
+            <!-- Passive sprocket rotate automatically according to the status of the active one -->
+            <xacro:if value="${mimic_enable}">
+                <mimic joint="wheel_${type}_joint" multiplier="1" offset="0"/>
+            </xacro:if>
         </joint>
         <link name="sprocket_${type}">
@@ -66,8 +70,4 @@
             <child link="wheel_${type}"/>
             <axis xyz="0 0 ${-1 * orientation}" />
-            <!-- Passive sprocket rotate automatically according to the status of the active one -->
-            <xacro:if value="${mimic_enable}">
-                <mimic joint="sprocket_${type}_joint" multiplier="1" offset="0"/>
-            </xacro:if>
         </joint>
         <link name="wheel_${type}">

File: src/tracked_robot_gazebo/urdf/diff_drive.gazebo.xacro (robot description, xacro)
@@ -7,8 +7,12 @@
             <!-- Plugin update rate in Hz -->
             <update_rate>${update_rate}</update_rate>
+            <num_wheel_pairs>2</num_wheel_pairs>
             <!-- Name of left joint, defaults to `left_joint` -->
             <left_joint>sprocket_left_joint</left_joint>
             <!-- Name of right joint, defaults to `right_joint` -->
             <right_joint>sprocket_right_joint</right_joint>
+            <left_joint>wheel_left_joint</left_joint>
+            <!-- Name of right joint, defaults to `right_joint` -->
+            <right_joint>wheel_right_joint</right_joint>
             <!-- The distance from the center of one wheel to the other, in meters, defaults to 0.34 m -->
             <wheel_separation>${wheel_separation}</wheel_separation>

File: src/tracked_robot_gazebo/urdf/tracked_robot.gazebo.xacro (robot description, xacro)
@@ -8,5 +8,5 @@
     <xacro:arg name="robot_name" default="tracked_robot" />
     <xacro:arg name="publish_odom_tf"  default="true"/>
-    <xacro:robot diff_drive_emulation="true" mimic_enable="false" path_meshes="file://$(find tracked_robot_description)/meshes"/>
+    <xacro:robot diff_drive_emulation="true" mimic_enable="true" path_meshes="file://$(find tracked_robot_description)/meshes"/>
     <!-- tracked_robot differential drive controller -->
     <xacro:track_drive parent="base_link"

Commit message: Fix URDF model

File: src/tracked_robot_description/urdf/track.urdf.xacro (robot description, xacro)
@@ -2,4 +2,12 @@
 <robot name="tracked_robot" xmlns:xacro="http://ros.org/wiki/xacro">
     <xacro:macro name="track" params="type parent radius diff_drive_emulation mimic_enable">
+        <xacro:macro name="cylinder_inertia" params="m r h">
+            <inertial>
+                <origin xyz="0 0 0" rpy="${pi/2} 0 0" />
+                <mass value="${m}" />
+                <inertia ixx="${(m/12) * (3*r*r + h*h)}" ixy="0" ixz="0" iyy="${(m/12) * (3*r*r + h*h)}"
+                    iyz="0" izz="${(m/2) * (r*r)}" />
+            </inertial>
+        </xacro:macro>
         <!-- Define orientation -->
         <xacro:if value="${type == 'left'}">
@@ -18,20 +26,15 @@
         <xacro:property name="scale" value="0.0046"/>
         <joint name="sprocket_${type}_joint" type="continuous">
-            <origin xyz="0.0 ${orientation * -0.235} -0.05" rpy="${orientation * M_PI/2} 0 0" />
+            <origin xyz="0.0 ${orientation * -0.235} -0.05" rpy="0 0 0" />
             <parent link="${parent}"/>
             <child link="sprocket_${type}"/>
-            <axis xyz="0 0 ${-1 * orientation}" />
+            <axis xyz="0 1 0" />
             <!-- Passive wheel rotate automatically according to the status of the active one -->
-            <xacro:if value="${mimic_enable}">
-                <mimic joint="wheel_${type}_joint" multiplier="1" offset="0"/>
-            </xacro:if>
+            <!-- <xacro:if value="${mimic_enable}">
+                <mimic joint="wheel_${type}_joint" multiplier="1" offset="0" />
+            </xacro:if> -->
         </joint>
         <link name="sprocket_${type}">
-         <inertial>
-            <mass value="1" />
-            <inertia ixx="0.0" ixy="0.0" ixz="0.0"
-                 iyy="0.0" iyz="0.0"
-                 izz="0.0" />
-        </inertial>
+            <xacro:cylinder_inertia m="0.1" r="${radius}" h="0.06" />
             <visual>
                 <origin xyz="0 0 0" rpy="0 0 0" />
@@ -44,5 +47,5 @@
             <!-- Collision cylinder -->
             <collision>
-                <origin xyz="0 0 0" rpy="0 0 0" />
+                <origin xyz="0 0 0" rpy="${pi/2} 0 0"/>
                 <geometry>
                     <cylinder length="0.06" radius="${radius}"/>

Commit message: fix robot model behavior

File: src/tracked_robot_description/urdf/track.urdf.xacro (robot description, xacro)
@@ -18,12 +18,8 @@
         <xacro:property name="scale" value="0.0046" />
         <joint name="sprocket_${type}_joint" type="continuous">
-            <origin xyz="0.0 ${orientation * -0.235} -0.05" rpy="${orientation * M_PI/2} 0 0" />
+            <origin xyz="0.0 ${orientation * -0.235} -0.05" rpy="0 0 0" />
             <parent link="${parent}" />
             <child link="sprocket_${type}" />
-            <axis xyz="0 0 ${-1 * orientation}" />
-            <!-- Passive wheel rotate automatically according to the status of the active one -->
-            <xacro:if value="${mimic_enable}">
-                <mimic joint="wheel_${type}_joint" multiplier="1" offset="0" />
-            </xacro:if>
+            <axis xyz="0 1 0" />
         </joint>
         <link name="sprocket_${type}">
@@ -35,5 +31,5 @@
             </inertial>
             <visual>
-                <origin xyz="0 0 0" rpy="0 0 0" />
+                <origin xyz="0 0 0" rpy="${pi/2} 0 0" />
                 <geometry>
                     <mesh filename="${path_meshes}/sprocket.stl" scale="${scale} ${scale} ${scale}" />
@@ -44,5 +40,5 @@
             <!-- Collision cylinder -->
             <collision>
-                <origin xyz="0 0 0" rpy="0 0 0" />
+                <origin xyz="0 0 0" rpy="${pi/2} 0 0" />
                 <geometry>
                     <cylinder length="0.06" radius="${radius}" />
@@ -55,6 +51,6 @@
             <kp>1e15</kp>
             <kd>1e13</kd>
-            <mu1>10000000</mu1>
-            <mu2>10000000</mu2>
+            <mu1>1000</mu1>
+            <mu2>1000</mu2>
             <!-- Ignition color reference -->
             <visual>
@@ -66,9 +62,10 @@
             </visual>
         </gazebo>
-        <joint name="wheel_${type}_joint" type="${mimic_type}">
-            <origin xyz="-0.221 ${orientation * -0.235} -0.05" rpy="${orientation * M_PI/2} 0 0" />
+        <joint name="wheel_${type}_joint" type="continuous">
+            <origin xyz="-0.221 ${orientation * -0.235} -0.05" rpy="0 0 0" />
             <parent link="${parent}" />
             <child link="wheel_${type}" />
-            <axis xyz="0 0 ${-1 * orientation}" />
+            <axis xyz="0 1 0" />
+            <mimic joint="sprocket_${type}_joint" multiplier="1" offset="0" />
         </joint>
         <link name="wheel_${type}">
@@ -80,5 +77,5 @@
             </inertial>
             <visual>
-                <origin xyz="0 0 0" rpy="0 0 0" />
+                <origin xyz="0 0 0" rpy="${pi/2} 0 0" />
                 <geometry>
                     <mesh filename="${path_meshes}/wheel.stl" scale="${scale} ${scale} ${scale}" />
@@ -89,5 +86,5 @@
             <!-- Collision cylinder -->
             <collision>
-                <origin xyz="0 0 0" rpy="0 0 0" />
+                <origin xyz="0 0 0" rpy="${pi/2} 0 0" />
                 <geometry>
                     <cylinder length="0.06" radius="${radius_wheel}" />
@@ -100,6 +97,6 @@
             <kp>1e15</kp>
             <kd>1e13</kd>
-            <mu1>0</mu1>
-            <mu2>0</mu2>
+            <mu1>1</mu1>
+            <mu2>1</mu2>
             <!-- Ignition color reference -->
             <visual>
@@ -111,9 +108,11 @@
             </visual>
         </gazebo>
-        <joint name="front_wheel_${type}_joint" type="${mimic_type}">
-            <origin xyz="0.221 ${orientation * -0.235} -0.05" rpy="${orientation * M_PI/2} 0 0" />
+        <joint name="front_wheel_${type}_joint" type="continuous">
+            <origin xyz="0.221 ${orientation * -0.235} -0.05" rpy="0 0 0" />
             <parent link="${parent}" />
             <child link="front_wheel_${type}" />
-            <axis xyz="0 0 ${-1 * orientation}" />
+            <axis xyz="0 1 0" />
+            <!-- Passive wheel rotate automatically according to the status of the active one -->
+            <mimic joint="sprocket_${type}_joint" multiplier="1" offset="0" />
         </joint>
         <link name="front_wheel_${type}">
@@ -125,5 +124,5 @@
             </inertial>
             <visual>
-                <origin xyz="0 0 0" rpy="0 0 0" />
+                <origin xyz="0 0 0" rpy="${pi/2} 0 0" />
                 <geometry>
                     <mesh filename="${path_meshes}/wheel.stl" scale="${scale} ${scale} ${scale}" />
@@ -134,5 +133,5 @@
             <!-- Collision cylinder -->
             <collision>
-                <origin xyz="0 0 0" rpy="0 0 0" />
+                <origin xyz="0 0 0" rpy="${pi/2} 0 0" />
                 <geometry>
                     <cylinder length="0.06" radius="${radius_wheel}" />
@@ -145,6 +144,6 @@
             <kp>1e15</kp>
             <kd>1e13</kd>
-            <mu1>0</mu1>
-            <mu2>0</mu2>
+            <mu1>1</mu1>
+            <mu2>1</mu2>
             <!-- Ignition color reference -->
             <visual>
@@ -156,5 +155,5 @@
             </visual>
         </gazebo>
-        <joint name="track_${type}_joint" type="continuous">
+        <joint name="track_${type}_joint" type="fixed">
             <origin xyz="0.0 ${orientation * -0.235} -0.05" rpy="0 0 0" />
             <parent link="${parent}" />
