Commit message: Add camera to gazebo

File: src/tracked_robot_description/urdf/camera.urdf.xacro (robot description, xacro)
@@ -3,5 +3,5 @@
     <xacro:macro name="camera"  params="parent">
         <joint name="camera_sensor_joint" type="fixed">
-            <origin xyz="0.6 0 -0.015" rpy="0 0 0"/>
+            <origin xyz="0.6 0 -0.015" rpy="0 ${M_PI/2} 0"/>
             <parent link="${parent}"/>
             <child link="camera_link"/>

File: src/tracked_robot_description/urdf/hand.urdf.xacro (robot description, xacro)
@@ -28,4 +28,5 @@
             <child link="hand"/>
             <axis xyz="0 0 1" />
+            <limit lower="-2" upper="2" effort="100" velocity="2"/>
         </joint>
         <link name="hand">

File: src/tracked_robot_gazebo/urdf/tracked_robot.gazebo.xacro (robot description, xacro)
@@ -4,4 +4,5 @@
     <!-- differential drive -->
     <xacro:include filename="$(find tracked_robot_gazebo)/urdf/diff_drive.gazebo.xacro"/>
+    <xacro:include filename="$(find tracked_robot_gazebo)/urdf/camera.gazebo.xacro"/>
     <xacro:arg name="robot_name" default="tracked_robot" />
     <xacro:arg name="publish_odom_tf"  default="true"/>
@@ -14,3 +15,5 @@
                        wheel_separation="0.4"
                        publish_odom_tf="$(arg publish_odom_tf)" />
+    <xacro:track_camera parent="camera_link"
+                        update_rate="100.0" />
 </robot>

Commit message: Hand plugin first implementation

File: src/tracked_robot_description/urdf/camera.urdf.xacro (robot description, xacro)
@@ -22,5 +22,5 @@
             </visual>
             <inertial>
-                <mass value="0.01"/>
+                <mass value="0.0001"/>
                 <origin rpy=" 0 0 0" xyz="0 0 0"/>
                 <inertia ixx="1.6666666666666668e-07" ixy="0" ixz="0" iyy="1.6666666666666668e-07" iyz="0" izz="1.6666666666666668e-07"/>

File: src/tracked_robot_description/urdf/hand.urdf.xacro (robot description, xacro)
@@ -11,5 +11,5 @@
         <link name="hand_base">
             <inertial>
-                <mass value="0.01"/>
+                <mass value="0.0001"/>
                 <origin rpy=" 0 0 0" xyz="0 0 0"/>
                 <inertia ixx="1.6666666666666668e-07" ixy="0" ixz="0" iyy="1.6666666666666668e-07" iyz="0" izz="1.6666666666666668e-07"/>
@@ -28,9 +28,8 @@
             <child link="hand"/>
             <axis xyz="0 0 1" />
-            <limit lower="-2" upper="2" effort="100" velocity="2"/>
         </joint>
         <link name="hand">
             <inertial>
-                <mass value="0.01"/>
+                <mass value="0.0001"/>
                 <origin rpy=" 0 0 0" xyz="0 0 0"/>
                 <inertia ixx="1.6666666666666668e-07" ixy="0" ixz="0" iyy="1.6666666666666668e-07" iyz="0" izz="1.6666666666666668e-07"/>

File: src/tracked_robot_description/urdf/track.urdf.xacro (robot description, xacro)
@@ -25,5 +25,5 @@
         <link name="sprocket_${type}">
             <inertial>
-                <mass value="0.01"/>
+                <mass value="0.001"/>
                 <origin rpy=" 0 0 0" xyz="0 0 0"/>
                 <inertia ixx="1.6666666666666668e-07" ixy="0" ixz="0" iyy="1.6666666666666668e-07" iyz="0" izz="1.6666666666666668e-07"/>
@@ -73,5 +73,5 @@
         <link name="wheel_${type}">
             <inertial>
-                <mass value="0.01"/>
+                <mass value="0.001"/>
                 <origin rpy=" 0 0 0" xyz="0 0 0"/>
                 <inertia ixx="1.6666666666666668e-07" ixy="0" ixz="0" iyy="1.6666666666666668e-07" iyz="0" izz="1.6666666666666668e-07"/>
@@ -116,5 +116,5 @@
         <link name="track_${type}">
             <inertial>
-                <mass value="0.01"/>
+                <mass value="0.001"/>
                 <origin rpy=" 0 0 0" xyz="0 0 0"/>
                 <inertia ixx="1.6666666666666668e-07" ixy="0" ixz="0" iyy="1.6666666666666668e-07" iyz="0" izz="1.6666666666666668e-07"/>

File: src/tracked_robot_description/urdf/tracked_robot_core.urdf.xacro (robot description, xacro)
@@ -28,4 +28,9 @@
     <xacro:macro name="robot" params="diff_drive_emulation mimic_enable:=true path_meshes:=package://tracked_robot_description/meshes">
     <link name="base_link">
+        <inertial>
+            <mass value="0.001"/>
+            <origin rpy=" 0 0 0" xyz="0 0 0"/>
+            <inertia ixx="1.6666666666666668e-07" ixy="0" ixz="0" iyy="1.6666666666666668e-07" iyz="0" izz="1.6666666666666668e-07"/>
+        </inertial>
         <visual>
             <origin xyz="0 0 -0.05" rpy="1.5707963267949 0 ${M_PI}"/>

File: src/tracked_robot_gazebo/urdf/tracked_robot.gazebo.xacro (robot description, xacro)
@@ -5,4 +5,5 @@
     <xacro:include filename="$(find tracked_robot_gazebo)/urdf/diff_drive.gazebo.xacro"/>
     <xacro:include filename="$(find tracked_robot_gazebo)/urdf/camera.gazebo.xacro"/>
+    <xacro:include filename="$(find tracked_robot_gazebo)/urdf/hand.gazebo.xacro"/>
     <xacro:arg name="robot_name" default="tracked_robot" />
     <xacro:arg name="publish_odom_tf"  default="true"/>
@@ -15,4 +16,5 @@
                        wheel_separation="0.4"
                        publish_odom_tf="$(arg publish_odom_tf)" />
+    <xacro:track_hand />
     <xacro:track_camera parent="camera_link"
                         update_rate="100.0" />

Commit message: add joystick support

File: src/tracked_robot_description/urdf/camera.urdf.xacro (robot description, xacro)
@@ -22,5 +22,5 @@
             </visual>
             <inertial>
-                <mass value="0.0001"/>
+                <mass value="0.001"/>
                 <origin rpy=" 0 0 0" xyz="0 0 0"/>
                 <inertia ixx="1.6666666666666668e-07" ixy="0" ixz="0" iyy="1.6666666666666668e-07" iyz="0" izz="1.6666666666666668e-07"/>

File: src/tracked_robot_description/urdf/hand.urdf.xacro (robot description, xacro)
@@ -11,5 +11,5 @@
         <link name="hand_base">
             <inertial>
-                <mass value="0.0001"/>
+                <mass value="0.001"/>
                 <origin rpy=" 0 0 0" xyz="0 0 0"/>
                 <inertia ixx="1.6666666666666668e-07" ixy="0" ixz="0" iyy="1.6666666666666668e-07" iyz="0" izz="1.6666666666666668e-07"/>
@@ -31,5 +31,5 @@
         <link name="hand">
             <inertial>
-                <mass value="0.0001"/>
+                <mass value="0.001"/>
                 <origin rpy=" 0 0 0" xyz="0 0 0"/>
                 <inertia ixx="1.6666666666666668e-07" ixy="0" ixz="0" iyy="1.6666666666666668e-07" iyz="0" izz="1.6666666666666668e-07"/>

File: src/tracked_robot_description/urdf/lidar.urdf.xacro (robot description, xacro)
@@ -22,5 +22,5 @@
             </visual>
             <inertial>
-                <mass value="0.0001"/>
+                <mass value="0.001"/>
                 <origin rpy=" 0 0 0" xyz="0 0 0"/>
                 <inertia ixx="1.6666666666666668e-07" ixy="0" ixz="0" iyy="1.6666666666666668e-07" iyz="0" izz="1.6666666666666668e-07"/>

File: src/tracked_robot_description/urdf/track.urdf.xacro (robot description, xacro)
@@ -29,5 +29,5 @@
         <link name="sprocket_${type}">
             <inertial>
-                <mass value="0.001"/>
+                <mass value="0.01"/>
                 <origin rpy=" 0 0 0" xyz="0 0 0"/>
                 <inertia ixx="1.6666666666666668e-07" ixy="0" ixz="0" iyy="1.6666666666666668e-07" iyz="0" izz="1.6666666666666668e-07"/>
@@ -73,5 +73,5 @@
         <link name="wheel_${type}">
             <inertial>
-                <mass value="0.001"/>
+                <mass value="0.01"/>
                 <origin rpy=" 0 0 0" xyz="0 0 0"/>
                 <inertia ixx="1.6666666666666668e-07" ixy="0" ixz="0" iyy="1.6666666666666668e-07" iyz="0" izz="1.6666666666666668e-07"/>
@@ -116,5 +116,5 @@
         <link name="track_${type}">
             <inertial>
-                <mass value="0.001"/>
+                <mass value="0.005"/>
                 <origin rpy=" 0 0 0" xyz="0 0 0"/>
                 <inertia ixx="1.6666666666666668e-07" ixy="0" ixz="0" iyy="1.6666666666666668e-07" iyz="0" izz="1.6666666666666668e-07"/>

File: src/tracked_robot_description/urdf/tracked_robot_core.urdf.xacro (robot description, xacro)
@@ -30,5 +30,5 @@
     <link name="base_link">
         <inertial>
-            <mass value="0.001"/>
+            <mass value="0.1"/>
             <origin rpy=" 0 0 0" xyz="0 0 0"/>
             <inertia ixx="1.6666666666666668e-07" ixy="0" ixz="0" iyy="1.6666666666666668e-07" iyz="0" izz="1.6666666666666668e-07"/>

Commit message: Fix navigation bringup

File: src/tracked_robot_description/urdf/camera.urdf.xacro (robot description, xacro)
@@ -11,9 +11,9 @@
             <origin xyz="0 0 0" rpy="0 0 0"/>
             <geometry>
-            <box size="0.1 0.1 0.1"/>
+                <box size="0.1 0.1 0.1"/>
             </geometry>
             </collision>
             <visual>
-            <origin xyz="0 0 0" rpy="0 0 0"/>
+                <origin xyz="0 0 0" rpy="0 0 0"/>
             <geometry>
                 <box size="0.02 0.02 0.02"/>

File: src/tracked_robot_description/urdf/track.urdf.xacro (robot description, xacro)
@@ -51,8 +51,4 @@
         </link>
         <gazebo reference="sprocket_${type}">
-            <kp>10000000</kp>
-            <kd>10000000</kd>
-            <mu1>10000000</mu1>
-            <mu2>10000000</mu2>
             <material>Gazebo/Blue</material>
             <!-- Ignition color reference -->
@@ -95,8 +91,4 @@
         </link>
         <gazebo reference="wheel_${type}">
-            <kp>10000000</kp>
-            <kd>10000000</kd>
-            <mu1>0</mu1>
-            <mu2>0</mu2>
             <material>Gazebo/Red</material>
             <!-- Ignition color reference -->

File: src/tracked_robot_gazebo/urdf/diff_drive.gazebo.xacro (robot description, xacro)
@@ -37,4 +37,16 @@
             <publis_wheel_joint_state>false</publis_wheel_joint_state>
             </plugin>
+            <plugin name="basic_mobile_bot_joint_state"
+            filename="libgazebo_ros_joint_state_publisher.so">
+            <ros>
+                <remapping>~/out:=joint_states</remapping>
+            </ros>
+            <update_rate>${update_rate}</update_rate>
+            <joint_name>sprocket_left_joint</joint_name>
+            <joint_name>sprocket_right_joint</joint_name>
+            <joint_name>wheel_left_joint</joint_name>
+            <joint_name>wheel_right_joint</joint_name>
+            <joint_name>hand_joint</joint_name>
+        </plugin>
         </gazebo>
     </xacro:macro>

File: src/tracked_robot_gazebo/urdf/lidar.gazebo.xacro (robot description, xacro)
@@ -28,7 +28,8 @@
             <plugin name="lidar_controller" filename="libgazebo_ros_ray_sensor.so" >
             <ros>
-                <remapping>~/out:=/scan</remapping>
+                <remapping>~/out:=scan</remapping>
             </ros>
             <output_type>sensor_msgs/LaserScan</output_type>
+            <frame_name>lidar_link</frame_name>
             </plugin>
         </sensor>

Commit message: Test static hand and fixing imu

File: src/tracked_robot_description/urdf/camera.urdf.xacro (robot description, xacro)
@@ -3,5 +3,5 @@
     <xacro:macro name="camera"  params="parent">
         <joint name="camera_sensor_joint" type="fixed">
-            <origin xyz="0.8 0 -0.015" rpy="0 ${M_PI/2} 0"/>
+            <origin xyz="0.6 0 -0.015" rpy="0 ${M_PI/2} 0"/>
             <parent link="${parent}"/>
             <child link="camera_link"/>

File: src/tracked_robot_description/urdf/hand.urdf.xacro (robot description, xacro)
@@ -10,9 +10,10 @@
         </joint>
         <link name="hand_base">
-            <inertial>
-                <mass value="0.001"/>
-                <origin rpy=" 0 0 0" xyz="0 0 0"/>
-                <inertia ixx="1.6666666666666668e-07" ixy="0" ixz="0" iyy="1.6666666666666668e-07" iyz="0" izz="1.6666666666666668e-07"/>
-            </inertial>
+        <inertial>
+            <mass value="2" />
+            <inertia ixx="1e-3" ixy="0.0" ixz="0.0"
+                 iyy="1e-3" iyz="0.0"
+                 izz="1e-3" />
+        </inertial>
             <visual>
                 <origin xyz="0 0 0" rpy="0 0 0"/>
@@ -23,5 +24,5 @@
             </visual>
         </link>
-       <joint name="hand_joint" type="continuous">
+       <joint name="hand_joint" type="fixed">
             <origin xyz="0 0 0.05" rpy="0 0 0" />
             <parent link="hand_base"/>
@@ -30,13 +31,8 @@
         </joint>
         <link name="hand">
-            <inertial>
-                <mass value="0.001"/>
-                <origin rpy=" 0 0 0" xyz="0 0 0"/>
-                <inertia ixx="1.6666666666666668e-07" ixy="0" ixz="0" iyy="1.6666666666666668e-07" iyz="0" izz="1.6666666666666668e-07"/>
-            </inertial>
             <visual>
-                <origin xyz="0.4 0 0" rpy="0 0 0"/>
+                <origin xyz="0.3     0 0" rpy="0 0 0"/>
                 <geometry>
-                     <box size="0.9 0.1 0.01"/>
+                     <box size="0.7 0.1 0.01"/>
                 </geometry>
                 <material name="Black" />

File: src/tracked_robot_description/urdf/track.urdf.xacro (robot description, xacro)
@@ -28,9 +28,10 @@
         </joint>
         <link name="sprocket_${type}">
-            <inertial>
-                <mass value="0.01"/>
-                <origin rpy=" 0 0 0" xyz="0 0 0"/>
-                <inertia ixx="1.6666666666666668e-07" ixy="0" ixz="0" iyy="1.6666666666666668e-07" iyz="0" izz="1.6666666666666668e-07"/>
-            </inertial>
+         <inertial>
+            <mass value="3" />
+            <inertia ixx="1e-3" ixy="0.0" ixz="0.0"
+                 iyy="1e-3" iyz="0.0"
+                 izz="1e-3" />
+        </inertial>
             <visual>
                 <origin xyz="0 0 0" rpy="0 0 0" />
@@ -72,9 +73,10 @@
         </joint>
         <link name="wheel_${type}">
-            <inertial>
-                <mass value="0.01"/>
-                <origin rpy=" 0 0 0" xyz="0 0 0"/>
-                <inertia ixx="1.6666666666666668e-07" ixy="0" ixz="0" iyy="1.6666666666666668e-07" iyz="0" izz="1.6666666666666668e-07"/>
-            </inertial>
+        <inertial>
+            <mass value="3" />
+            <inertia ixx="1e-3" ixy="0.0" ixz="0.0"
+                 iyy="1e-3" iyz="0.0"
+                 izz="1e-3" />
+        </inertial>
             <visual>
                 <origin xyz="0 0 0" rpy="0 0 0" />
@@ -115,9 +117,4 @@
         </joint>
         <link name="track_${type}">
-            <inertial>
-                <mass value="0.005"/>
-                <origin rpy=" 0 0 0" xyz="0 0 0"/>
-                <inertia ixx="1.6666666666666668e-07" ixy="0" ixz="0" iyy="1.6666666666666668e-07" iyz="0" izz="1.6666666666666668e-07"/>
-            </inertial>
             <visual>
                 <origin xyz="0 0 0" rpy="${M_PI/2} 0 0" />

File: src/tracked_robot_description/urdf/tracked_robot_core.urdf.xacro (robot description, xacro)
@@ -37,9 +37,4 @@
   </joint>
     <link name="base_link">
-        <inertial>
-            <mass value="0.1"/>
-            <origin rpy=" 0 0 0" xyz="0 0 0"/>
-            <inertia ixx="1.6666666666666668e-07" ixy="0" ixz="0" iyy="1.6666666666666668e-07" iyz="0" izz="1.6666666666666668e-07"/>
-        </inertial>
         <visual>
             <origin xyz="0 0 -0.05" rpy="1.5707963267949 0 ${M_PI}"/>

File: src/tracked_robot_gazebo/urdf/diff_drive.gazebo.xacro (robot description, xacro)
@@ -47,5 +47,4 @@
             <joint_name>wheel_left_joint</joint_name>
             <joint_name>wheel_right_joint</joint_name>
-            <joint_name>hand_joint</joint_name>
         </plugin>
         </gazebo>

File: src/tracked_robot_gazebo/urdf/imu.gazebo.xacro (robot description, xacro)
@@ -10,62 +10,11 @@
         </ros>
         <initial_orientation_as_reference>false</initial_orientation_as_reference>
+        <bodyName>imu_link</bodyName>
+        <updateRateHZ>10.0</updateRateHZ>
+        <gaussianNoise>0.0</gaussianNoise>
+        <xyzOffset>0 0 0</xyzOffset>
+        <rpyOffset>0 0 0</rpyOffset>
+        <frameName>imu_link</frameName>
       </plugin>
-      <always_on>true</always_on>
-      <update_rate>100</update_rate>
-      <visualize>true</visualize>
-      <imu>
-        <angular_velocity>
-          <x>
-            <noise type="gaussian">
-              <mean>0.0</mean>
-              <stddev>2e-4</stddev>
-              <bias_mean>0.0000075</bias_mean>
-              <bias_stddev>0.0000008</bias_stddev>
-            </noise>
-          </x>
-          <y>
-            <noise type="gaussian">
-              <mean>0.0</mean>
-              <stddev>2e-4</stddev>
-              <bias_mean>0.0000075</bias_mean>
-              <bias_stddev>0.0000008</bias_stddev>
-            </noise>
-          </y>
-          <z>
-            <noise type="gaussian">
-              <mean>0.0</mean>
-              <stddev>2e-4</stddev>
-              <bias_mean>0.0000075</bias_mean>
-              <bias_stddev>0.0000008</bias_stddev>
-            </noise>
-          </z>
-        </angular_velocity>
-        <linear_acceleration>
-          <x>
-            <noise type="gaussian">
-              <mean>0.0</mean>
-              <stddev>1.7e-2</stddev>
-              <bias_mean>0.1</bias_mean>
-              <bias_stddev>0.001</bias_stddev>
-            </noise>
-          </x>
-          <y>
-            <noise type="gaussian">
-              <mean>0.0</mean>
-              <stddev>1.7e-2</stddev>
-              <bias_mean>0.1</bias_mean>
-              <bias_stddev>0.001</bias_stddev>
-            </noise>
-          </y>
-          <z>
-            <noise type="gaussian">
-              <mean>0.0</mean>
-              <stddev>1.7e-2</stddev>
-              <bias_mean>0.1</bias_mean>
-              <bias_stddev>0.001</bias_stddev>
-            </noise>
-          </z>
-        </linear_acceleration>
-      </imu>
     </sensor>
   </gazebo>

File: src/tracked_robot_gazebo/urdf/tracked_robot.gazebo.xacro (robot description, xacro)
@@ -6,5 +6,4 @@
     <xacro:include filename="$(find tracked_robot_gazebo)/urdf/camera.gazebo.xacro"/>
     <xacro:include filename="$(find tracked_robot_gazebo)/urdf/lidar.gazebo.xacro"/>
-    <xacro:include filename="$(find tracked_robot_gazebo)/urdf/hand.gazebo.xacro"/>
     <xacro:include filename="$(find tracked_robot_gazebo)/urdf/imu.gazebo.xacro"/>
     <xacro:arg name="robot_name" default="tracked_robot" />
@@ -18,5 +17,4 @@
                        wheel_separation="0.4"
                        publish_odom_tf="$(arg publish_odom_tf)" />
-    <xacro:track_hand />
     <xacro:track_camera parent="camera_link"
                         update_rate="30.0" />
