Commit message: hardware changes

File: src/tracked_robot_description/urdf/camera.urdf.xacro (robot description, xacro)
@@ -3,5 +3,5 @@
     <xacro:macro name="camera"  params="parent">
         <joint name="camera_sensor_joint" type="fixed">
-            <origin xyz="0.8 0 -0.015" rpy="0 ${M_PI/2} 0"/>
+            <origin xyz="0.6 0 -0.015" rpy="0 ${M_PI/2} 0"/>
             <parent link="${parent}"/>
             <child link="camera_link"/>
@@ -11,9 +11,9 @@
             <origin xyz="0 0 0" rpy="0 0 0"/>
             <geometry>
-            <box size="0.1 0.1 0.1"/>
+                <box size="0.1 0.1 0.1"/>
             </geometry>
             </collision>
             <visual>
-            <origin xyz="0 0 0" rpy="0 0 0"/>
+                <origin xyz="0 0 0" rpy="0 0 0"/>
             <geometry>
                 <box size="0.02 0.02 0.02"/>

File: src/tracked_robot_description/urdf/lidar.urdf.xacro (robot description, xacro)
@@ -19,5 +19,5 @@
                 <cylinder radius="0.05" length="0.04"/>
             </geometry>
-            <material name="red"/>
+            <!--material name="red"/-->
             </visual>
             <inertial>

File: src/tracked_robot_description/urdf/track.urdf.xacro (robot description, xacro)
@@ -18,5 +18,5 @@
         <xacro:property name="scale" value="0.0046"/>
         <joint name="sprocket_${type}_joint" type="continuous">
-            <origin xyz="0.221 ${orientation * -0.235} -0.05" rpy="${orientation * M_PI/2} 0 0" />
+            <origin xyz="0.0 ${orientation * -0.235} -0.05" rpy="${orientation * M_PI/2} 0 0" />
             <parent link="${parent}"/>
             <child link="sprocket_${type}"/>
@@ -28,9 +28,10 @@
         </joint>
         <link name="sprocket_${type}">
-            <inertial>
-                <mass value="0.01"/>
-                <origin rpy=" 0 0 0" xyz="0 0 0"/>
-                <inertia ixx="1.6666666666666668e-07" ixy="0" ixz="0" iyy="1.6666666666666668e-07" iyz="0" izz="1.6666666666666668e-07"/>
-            </inertial>
+         <inertial>
+            <mass value="3" />
+            <inertia ixx="1e-3" ixy="0.0" ixz="0.0"
+                 iyy="1e-3" iyz="0.0"
+                 izz="1e-3" />
+        </inertial>
             <visual>
                 <origin xyz="0 0 0" rpy="0 0 0" />
@@ -51,9 +52,9 @@
         </link>
         <gazebo reference="sprocket_${type}">
+            <material>Gazebo/Blue</material>
             <kp>10000000</kp>
             <kd>10000000</kd>
             <mu1>10000000</mu1>
             <mu2>10000000</mu2>
-            <material>Gazebo/Blue</material>
             <!-- Ignition color reference -->
             <visual>
@@ -66,5 +67,5 @@
         </gazebo>
         <joint name="wheel_${type}_joint" type="${mimic_type}">
-            <origin xyz="-0.221 ${orientation * -0.235} -0.05" rpy="${orientation * M_PI/2} 0 0" />
+            <origin xyz="-0.442 ${orientation * -0.235} -0.05" rpy="${orientation * M_PI/2} 0 0" />
             <parent link="${parent}"/>
             <child link="wheel_${type}"/>
@@ -72,9 +73,10 @@
         </joint>
         <link name="wheel_${type}">
-            <inertial>
-                <mass value="0.01"/>
-                <origin rpy=" 0 0 0" xyz="0 0 0"/>
-                <inertia ixx="1.6666666666666668e-07" ixy="0" ixz="0" iyy="1.6666666666666668e-07" iyz="0" izz="1.6666666666666668e-07"/>
-            </inertial>
+        <inertial>
+            <mass value="3" />
+            <inertia ixx="1e-3" ixy="0.0" ixz="0.0"
+                 iyy="1e-3" iyz="0.0"
+                 izz="1e-3" />
+        </inertial>
             <visual>
                 <origin xyz="0 0 0" rpy="0 0 0" />
@@ -95,9 +97,9 @@
         </link>
         <gazebo reference="wheel_${type}">
+            <material>Gazebo/Red</material>
             <kp>10000000</kp>
             <kd>10000000</kd>
             <mu1>0</mu1>
             <mu2>0</mu2>
-            <material>Gazebo/Red</material>
             <!-- Ignition color reference -->
             <visual>
@@ -110,14 +112,9 @@
         </gazebo>
         <joint name="track_${type}_joint" type="fixed">
-            <origin xyz="0.0 ${orientation * -0.235} -0.05" rpy="${orientation * M_PI/2} 0 0" />
+            <origin xyz="-0.221 ${orientation * -0.235} -0.05" rpy="${orientation * M_PI/2} 0 0" />
             <parent link="${parent}"/>
             <child link="track_${type}"/>
         </joint>
         <link name="track_${type}">
-            <inertial>
-                <mass value="0.005"/>
-                <origin rpy=" 0 0 0" xyz="0 0 0"/>
-                <inertia ixx="1.6666666666666668e-07" ixy="0" ixz="0" iyy="1.6666666666666668e-07" iyz="0" izz="1.6666666666666668e-07"/>
-            </inertial>
             <visual>
                 <origin xyz="0 0 0" rpy="${M_PI/2} 0 0" />

File: src/tracked_robot_description/urdf/tracked_robot_core.urdf.xacro (robot description, xacro)
@@ -1,7 +1,11 @@
 <?xml version="1.0" ?>
 <robot name="tracked_robot" xmlns:xacro="http://ros.org/wiki/xacro">
+    <xacro:arg name="use_ros2_control" default="true"/>
+    <xacro:arg name="sim_mode" default="false"/>
     <xacro:include filename="track.urdf.xacro" />
     <xacro:include filename="hand.urdf.xacro" />
     <xacro:include filename="lidar.urdf.xacro" />
+    <xacro:include filename="imu.urdf.xacro" />
+    <xacro:include filename="gps.urdf.xacro" />
     <material name="Black">
         <color rgba="0.1 0.1 0.1 1.0"/>
@@ -26,14 +30,16 @@
     </material>
     <xacro:property name="M_PI" value="3.14159"/>
-    <xacro:property name="sprocket_radius" value="0.06"/>
+    <xacro:property name="sprocket_radius" value="0.02545"/>
     <xacro:macro name="robot" params="diff_drive_emulation mimic_enable:=true path_meshes:=package://tracked_robot_description/meshes">
+<link name="base_footprint"/>
+    <!-- The base footprint of the robot is located underneath the chassis -->
+    <joint name="base_joint" type="fixed">
+        <parent link="base_footprint"/>
+        <child link="base_link" />
+        <origin xyz="0.0 0.0 0.1" rpy="0 0 0"/>
+    </joint>
     <link name="base_link">
-        <inertial>
-            <mass value="0.1"/>
-            <origin rpy=" 0 0 0" xyz="0 0 0"/>
-            <inertia ixx="1.6666666666666668e-07" ixy="0" ixz="0" iyy="1.6666666666666668e-07" iyz="0" izz="1.6666666666666668e-07"/>
-        </inertial>
         <visual>
-            <origin xyz="0 0 -0.05" rpy="1.5707963267949 0 ${M_PI}"/>
+            <origin xyz="-0.221 0 -0.05" rpy="1.5707963267949 0 ${M_PI}"/>
             <geometry>
                 <mesh filename="${path_meshes}/robot_base.stl" scale="1 1 1" />
@@ -46,4 +52,5 @@
     <xacro:hand parent="base_link" />
     <xacro:lidar parent="base_link" />
+    <xacro:imu parent="base_link" />
     </xacro:macro>
 </robot>

File: src/tracked_robot_gazebo/urdf/diff_drive.gazebo.xacro (robot description, xacro)
@@ -5,35 +5,43 @@
         <gazebo>
             <plugin filename="libgazebo_ros_diff_drive.so" name="skid_steer_drive_controller">
-            <!-- Plugin update rate in Hz -->
-            <update_rate>${update_rate}</update_rate>
-            <num_wheel_pairs>2</num_wheel_pairs>
-            <!-- Name of left joint, defaults to `left_joint` -->
-            <left_joint>sprocket_left_joint</left_joint>
-            <!-- Name of right joint, defaults to `right_joint` -->
-            <right_joint>sprocket_right_joint</right_joint>
-            <left_joint>wheel_left_joint</left_joint>
-            <!-- Name of right joint, defaults to `right_joint` -->
-            <right_joint>wheel_right_joint</right_joint>
-            <!-- The distance from the center of one wheel to the other, in meters, defaults to 0.34 m -->
-            <wheel_separation>${wheel_separation}</wheel_separation>
-            <!-- Diameter of the wheels, in meters, defaults to 0.15 m -->
-            <wheel_diameter>${wheel_radius * 2}</wheel_diameter>
-            <!-- Wheel acceleration, in rad/s^2, defaults to 0.0 rad/s^2 -->
-            <wheel_acceleration>0.0</wheel_acceleration>
-            <!-- Maximum torque which the wheels can produce, in Nm, defaults to 5 Nm -->
-            <max_wheel_torque>15</max_wheel_torque>
-            <!-- Odometry frame, defaults to `odom` -->
-            <odometry_frame>odom</odometry_frame>
-            <!-- Robot frame to calculate odometry from, defaults to `base_footprint` -->
-            <robot_base_frame>${parent}</robot_base_frame>
-            <!-- Set to true to publish transforms for the odometry, defaults to true -->
-            <publish_odom>true</publish_odom>
-            <publish_odom_tf>${publish_odom_tf}</publish_odom_tf>
-            <!-- Set to true to publish transforms for the wheel links, defaults to false -->
-            <publish_wheel_tf>true</publish_wheel_tf>
-            <!-- Odometry source, 0 for ENCODER, 1 for WORLD, defaults to WORLD -->
-            <odometry_source>1</odometry_source>
-            <!-- Set to true to publish sensor_msgs/JointState on /joint_states for the wheel joints, defaults to false -->
-            <publis_wheel_joint_state>false</publis_wheel_joint_state>
+                <!--ros>
+                    <namespace>/example</namespace>
+                </ros-->
+                <!-- Plugin update rate in Hz -->
+                <update_rate>${update_rate}</update_rate>
+                <num_wheel_pairs>2</num_wheel_pairs>
+                <!-- Name of left joint, defaults to `left_joint` -->
+                <left_joint>sprocket_left_joint</left_joint>
+                <!-- Name of right joint, defaults to `right_joint` -->
+                <right_joint>sprocket_right_joint</right_joint>
+                <left_joint>wheel_left_joint</left_joint>
+                <!-- Name of right joint, defaults to `right_joint` -->
+                <right_joint>wheel_right_joint</right_joint>
+                <!-- The distance from the center of one wheel to the other, in meters, defaults to 0.34 m -->
+                <wheel_separation>${wheel_separation}</wheel_separation>
+                <!-- Diameter of the wheels, in meters, defaults to 0.15 m -->
+                <wheel_diameter>${wheel_radius * 2}</wheel_diameter>
+                <!-- Wheel acceleration, in rad/s^2, defaults to 0.0 rad/s^2 -->
+                <wheel_acceleration>0.0</wheel_acceleration>
+                <!-- Maximum torque which the wheels can produce, in Nm, defaults to 5 Nm -->
+                <max_wheel_torque>15</max_wheel_torque>
+                <!-- Odometry frame, defaults to `odom` -->
+                <!--odometry_frame>odom</odometry_frame-->
+                <!-- Robot frame to calculate odometry from, defaults to `base_footprint` -->
+                <robot_base_frame>${parent}</robot_base_frame>
+                <!-- Set to true to publish transforms for the odometry, defaults to true -->
+                <publish_odom>true</publish_odom>
+                <publish_odom_tf>false</publish_odom_tf>
+                <!-- Set to true to publish transforms for the wheel links, defaults to false -->
+                <publish_wheel_tf>true</publish_wheel_tf>
+                <!-- Odometry source, 0 for ENCODER, 1 for WORLD, defaults to WORLD -->
+                <!--odometry_source>0</odometry_source-->
+                <odometry_frame>odom</odometry_frame>
+                <!-- Set to true to publish sensor_msgs/JointState on /joint_states for the wheel joints, defaults to false -->
+                <publis_wheel_joint_state>false</publis_wheel_joint_state>
+                <!-- Change the ROS topic we will publish the odometry data to -->
+                <ros>
+                    <remapping>odom:=example/odom</remapping>
+                </ros>
             </plugin>
         </gazebo>

File: src/tracked_robot_gazebo/urdf/tracked_robot.gazebo.xacro (robot description, xacro)
@@ -7,9 +7,11 @@
     <xacro:include filename="$(find tracked_robot_gazebo)/urdf/lidar.gazebo.xacro"/>
     <xacro:include filename="$(find tracked_robot_gazebo)/urdf/hand.gazebo.xacro"/>
+    <xacro:include filename="$(find tracked_robot_gazebo)/urdf/imu.gazebo.xacro"/>
+    <xacro:include filename="$(find tracked_robot_gazebo)/urdf/gps.gazebo.xacro"/>
     <xacro:arg name="robot_name" default="tracked_robot" />
     <xacro:arg name="publish_odom_tf"  default="true"/>
     <xacro:robot diff_drive_emulation="true" mimic_enable="true" path_meshes="file://$(find tracked_robot_description)/meshes"/>
     <!-- tracked_robot differential drive controller -->
-    <xacro:track_drive parent="base_link"
+    <xacro:track_drive parent="base_footptint"
                        robot_name="$(arg robot_name)"
                        update_rate="100.0"
@@ -18,4 +20,6 @@
                        publish_odom_tf="$(arg publish_odom_tf)" />
     <xacro:track_hand />
+    <xacro:track_gps parent="gps_link"/>
+    <xacro:track_imu parent="imu_link"/>
     <xacro:track_camera parent="camera_link"
                         update_rate="100.0" />

Commit message: Avoid mines on the field

File: src/tracked_robot_description/urdf/camera.urdf.xacro (robot description, xacro)
@@ -3,5 +3,5 @@
     <xacro:macro name="camera"  params="parent">
         <joint name="camera_sensor_joint" type="fixed">
-            <origin xyz="0.6 0 -0.015" rpy="0 ${M_PI/2} 0"/>
+            <origin xyz="0.6 0 -0.030" rpy="0 ${M_PI/2} 0"/>
             <parent link="${parent}"/>
             <child link="camera_link"/>

File: src/tracked_robot_description/urdf/hand.urdf.xacro (robot description, xacro)
@@ -19,5 +19,5 @@
                 <origin xyz="0 0 0" rpy="0 0 0"/>
                 <geometry>
-                     <cylinder length="0.18" radius="0.06"/>
+                     <cylinder length="0.36" radius="0.06"/>
                 </geometry>
                 <material name="Black" />
@@ -25,5 +25,5 @@
         </link>
        <joint name="hand_joint" type="fixed">
-            <origin xyz="0 0 0.09" rpy="0 0 0" />
+            <origin xyz="0 0 0.18" rpy="0 0 0" />
             <parent link="hand_base"/>
             <child link="hand"/>
