Commit message: Fix robot rotation center

File: src/tracked_robot_description/urdf/camera.urdf.xacro (robot description, xacro)
@@ -1,28 +1,29 @@
 <?xml version="1.0"?>
 <robot name="tracked_robot" xmlns:xacro="http://ros.org/wiki/xacro">
-    <xacro:macro name="camera"  params="parent">
+    <xacro:macro name="camera" params="parent">
         <joint name="camera_sensor_joint" type="fixed">
-            <origin xyz="0.6 0 -0.030" rpy="0 ${M_PI/2} 0"/>
-            <parent link="${parent}"/>
-            <child link="camera_link"/>
+            <origin xyz="0.6 0 -0.030" rpy="0 ${M_PI/2} 0" />
+            <parent link="${parent}" />
+            <child link="camera_link" />
         </joint>
         <link name="camera_link">
             <collision>
-            <origin xyz="0 0 0" rpy="0 0 0"/>
-            <geometry>
-                <box size="0.1 0.1 0.1"/>
-            </geometry>
+                <origin xyz="0 0 0" rpy="0 0 0" />
+                <geometry>
+                    <box size="0.1 0.1 0.1" />
+                </geometry>
             </collision>
             <visual>
-                <origin xyz="0 0 0" rpy="0 0 0"/>
-            <geometry>
-                <box size="0.02 0.02 0.02"/>
-            </geometry>
-            <material name="Red"/>
+                <origin xyz="0 0 0" rpy="0 0 0" />
+                <geometry>
+                    <box size="0.02 0.02 0.02" />
+                </geometry>
+                <material name="Red" />
             </visual>
             <inertial>
-                <mass value="0.001"/>
-                <origin rpy=" 0 0 0" xyz="0 0 0"/>
-                <inertia ixx="1.6666666666666668e-07" ixy="0" ixz="0" iyy="1.6666666666666668e-07" iyz="0" izz="1.6666666666666668e-07"/>
+                <mass value="0.001" />
+                <origin rpy=" 0 0 0" xyz="0 0 0" />
+                <inertia ixx="1.6666666666666668e-07" ixy="0" ixz="0" iyy="1.6666666666666668e-07"
+                    iyz="0" izz="1.6666666666666668e-07" />
             </inertial>
         </link>

File: src/tracked_robot_description/urdf/gps.urdf.xacro (robot description, xacro)
@@ -1,28 +1,29 @@
 <?xml version="1.0"?>
 <robot name="tracked_robot" xmlns:xacro="http://ros.org/wiki/xacro">
-    <xacro:macro name="gps"  params="parent">
+    <xacro:macro name="gps" params="parent">
         <joint name="gps_sensor_joint" type="fixed">
-            <origin xyz="0 0 0" rpy="0 0 0"/>
-            <parent link="${parent}"/>
-            <child link="gps_link"/>
+            <origin xyz="0 0 0" rpy="0 0 0" />
+            <parent link="${parent}" />
+            <child link="gps_link" />
         </joint>
         <link name="gps_link">
             <collision>
-            <origin xyz="0 0 0" rpy="0 0 0"/>
-            <geometry>
-            <box size="0.1 0.1 0.1"/>
-            </geometry>
+                <origin xyz="0 0 0" rpy="0 0 0" />
+                <geometry>
+                    <box size="0.1 0.1 0.1" />
+                </geometry>
             </collision>
             <visual>
-            <origin xyz="0 0 0" rpy="0 0 0"/>
-            <geometry>
-                <box size="0.02 0.02 0.02"/>
-            </geometry>
-            <material name="Red"/>
+                <origin xyz="0 0 0" rpy="0 0 0" />
+                <geometry>
+                    <box size="0.02 0.02 0.02" />
+                </geometry>
+                <material name="Red" />
             </visual>
             <inertial>
-                <mass value="0.001"/>
-                <origin rpy=" 0 0 0" xyz="0 0 0"/>
-                <inertia ixx="1.6666666666666668e-07" ixy="0" ixz="0" iyy="1.6666666666666668e-07" iyz="0" izz="1.6666666666666668e-07"/>
+                <mass value="0.001" />
+                <origin rpy=" 0 0 0" xyz="0 0 0" />
+                <inertia ixx="1.6666666666666668e-07" ixy="0" ixz="0" iyy="1.6666666666666668e-07"
+                    iyz="0" izz="1.6666666666666668e-07" />
             </inertial>
         </link>

File: src/tracked_robot_description/urdf/imu.urdf.xacro (robot description, xacro)
@@ -1,28 +1,29 @@
 <?xml version="1.0"?>
 <robot name="tracked_robot" xmlns:xacro="http://ros.org/wiki/xacro">
-    <xacro:macro name="imu"  params="parent">
+    <xacro:macro name="imu" params="parent">
         <joint name="imu_sensor_joint" type="fixed">
-            <origin xyz="0 0 0" rpy="0 0 0"/>
-            <parent link="${parent}"/>
-            <child link="imu_link"/>
+            <origin xyz="0 0 0" rpy="0 0 0" />
+            <parent link="${parent}" />
+            <child link="imu_link" />
         </joint>
         <link name="imu_link">
             <collision>
-            <origin xyz="0 0 0" rpy="0 0 0"/>
-            <geometry>
-            <box size="0.1 0.1 0.1"/>
-            </geometry>
+                <origin xyz="0 0 0" rpy="0 0 0" />
+                <geometry>
+                    <box size="0.1 0.1 0.1" />
+                </geometry>
             </collision>
             <visual>
-            <origin xyz="0 0 0" rpy="0 0 0"/>
-            <geometry>
-                <box size="0.02 0.02 0.02"/>
-            </geometry>
-            <material name="Red"/>
+                <origin xyz="0 0 0" rpy="0 0 0" />
+                <geometry>
+                    <box size="0.02 0.02 0.02" />
+                </geometry>
+                <material name="Red" />
             </visual>
             <inertial>
-                <mass value="0.001"/>
-                <origin rpy=" 0 0 0" xyz="0 0 0"/>
-                <inertia ixx="1.6666666666666668e-07" ixy="0" ixz="0" iyy="1.6666666666666668e-07" iyz="0" izz="1.6666666666666668e-07"/>
+                <mass value="0.001" />
+                <origin rpy=" 0 0 0" xyz="0 0 0" />
+                <inertia ixx="1.6666666666666668e-07" ixy="0" ixz="0" iyy="1.6666666666666668e-07"
+                    iyz="0" izz="1.6666666666666668e-07" />
             </inertial>
         </link>

File: src/tracked_robot_description/urdf/lidar.urdf.xacro (robot description, xacro)
@@ -1,28 +1,29 @@
 <?xml version="1.0"?>
 <robot name="tracked_robot" xmlns:xacro="http://ros.org/wiki/xacro">
-    <xacro:macro name="lidar"  params="parent">
+    <xacro:macro name="lidar" params="parent">
         <joint name="lidar_sensor_joint" type="fixed">
             <origin xyz="0.0 0 0.11" rpy="0 0 0" />
-            <parent link="${parent}"/>
-            <child link="lidar_link"/>
+            <parent link="${parent}" />
+            <child link="lidar_link" />
         </joint>
         <link name="lidar_link">
             <collision>
-            <origin xyz="0 0 0" rpy="0 0 0"/>
-            <geometry>
-                <cylinder radius="0.05" length="0.04"/>
-            </geometry>
+                <origin xyz="0 0 0" rpy="0 0 0" />
+                <geometry>
+                    <cylinder radius="0.05" length="0.04" />
+                </geometry>
             </collision>
             <visual>
-            <origin xyz="0 0 0" rpy="0 0 0"/>
-            <geometry>
-                <cylinder radius="0.05" length="0.04"/>
-            </geometry>
-            <material name="red"/>
+                <origin xyz="0 0 0" rpy="0 0 0" />
+                <geometry>
+                    <cylinder radius="0.05" length="0.04" />
+                </geometry>
+                <material name="Red" />
             </visual>
             <inertial>
-                <mass value="0.001"/>
-                <origin rpy=" 0 0 0" xyz="0 0 0"/>
-                <inertia ixx="1.6666666666666668e-07" ixy="0" ixz="0" iyy="1.6666666666666668e-07" iyz="0" izz="1.6666666666666668e-07"/>
+                <mass value="0.001" />
+                <origin rpy=" 0 0 0" xyz="0 0 0" />
+                <inertia ixx="1.6666666666666668e-07" ixy="0" ixz="0" iyy="1.6666666666666668e-07"
+                    iyz="0" izz="1.6666666666666668e-07" />
             </inertial>
         </link>

File: src/tracked_robot_description/urdf/track.urdf.xacro (robot description, xacro)
@@ -4,39 +4,39 @@
         <!-- Define orientation -->
         <xacro:if value="${type == 'left'}">
-            <xacro:property name="orientation" value="-1"/>
+            <xacro:property name="orientation" value="-1" />
         </xacro:if>
         <xacro:if value="${type == 'right'}">
-            <xacro:property name="orientation" value="1"/>
+            <xacro:property name="orientation" value="1" />
         </xacro:if>
         <xacro:if value="${mimic_enable}">
-            <xacro:property name="mimic_type" value="continuous"/>
+            <xacro:property name="mimic_type" value="continuous" />
         </xacro:if>
         <xacro:unless value="${mimic_enable}">
-            <xacro:property name="mimic_type" value="fixed"/>
+            <xacro:property name="mimic_type" value="fixed" />
         </xacro:unless>
-        <xacro:property name="radius_wheel" value="${radius}"/>
-        <xacro:property name="scale" value="0.0046"/>
-        <joint name="sprocket_${type}_joint" type="continuous">
-            <origin xyz="0.0 ${orientation * -0.235} -0.05" rpy="${orientation * M_PI/2} 0 0" />
-            <parent link="${parent}"/>
-            <child link="sprocket_${type}"/>
+        <xacro:property name="radius_wheel" value="${radius}" />
+        <xacro:property name="scale" value="0.0046" />
+        <joint name="sprocket_${type}_joint" type="${mimic_type}">
+            <origin xyz="0.221 ${orientation * -0.235} -0.05" rpy="${orientation * M_PI/2} 0 0" />
+            <parent link="${parent}" />
+            <child link="sprocket_${type}" />
             <axis xyz="0 0 ${-1 * orientation}" />
             <!-- Passive wheel rotate automatically according to the status of the active one -->
             <xacro:if value="${mimic_enable}">
-                <mimic joint="wheel_${type}_joint" multiplier="1" offset="0"/>
+                <mimic joint="wheel_${type}_joint" multiplier="1" offset="0" />
             </xacro:if>
         </joint>
         <link name="sprocket_${type}">
-         <inertial>
-            <mass value="3" />
-            <inertia ixx="1e-3" ixy="0.0" ixz="0.0"
-                 iyy="1e-3" iyz="0.0"
-                 izz="1e-3" />
-        </inertial>
+            <inertial>
+                <mass value="3" />
+                <inertia ixx="1e-3" ixy="0.0" ixz="0.0"
+                    iyy="1e-3" iyz="0.0"
+                    izz="1e-3" />
+            </inertial>
             <visual>
                 <origin xyz="0 0 0" rpy="0 0 0" />
                 <geometry>
-                    <mesh filename="${path_meshes}/sprocket.stl" scale="${scale} ${scale} ${scale}"/>
-                    <cylinder length="0.06" radius="${radius_wheel}"/>
+                    <mesh filename="${path_meshes}/sprocket.stl" scale="${scale} ${scale} ${scale}" />
+                    <cylinder length="0.06" radius="${radius_wheel}" />
                 </geometry>
                 <material name="Black" />
@@ -46,5 +46,69 @@
                 <origin xyz="0 0 0" rpy="0 0 0" />
                 <geometry>
-                    <cylinder length="0.06" radius="${radius}"/>
+                    <cylinder length="0.06" radius="${radius}" />
+                </geometry>
+                <material name="Black" />
+            </collision>
+        </link>
+        <joint name="drive_${type}_joint" type="continuous">
+            <origin xyz="0.0 ${orientation * -0.235} -0.05" rpy="${orientation * M_PI/2} 0 0" />
+            <parent link="${parent}" />
+            <child link="drive_${type}" />
+            <axis xyz="0 0 ${-1 * orientation}" />
+            <xacro:if value="${mimic_enable}">
+                <mimic joint="sprocket_${type}_joint" multiplier="1" offset="0" />
+            </xacro:if>
+            <!-- Passive wheel rotate automatically according to the status of the active one -->
+        </joint>
+        <link name="drive_${type}">
+            <inertial>
+                <mass value="3" />
+                <inertia ixx="1e-3" ixy="0.0" ixz="0.0"
+                    iyy="1e-3" iyz="0.0"
+                    izz="1e-3" />
+            </inertial>
+            <visual>
+                <origin xyz="0 0 0" rpy="0 0 0" />
+                <geometry>
+                    <mesh filename="${path_meshes}/sprocket.stl" scale="${scale} ${scale} ${scale}" />
+                    <cylinder length="0.06" radius="${radius_wheel}" />
+                </geometry>
+                <material name="Black" />
+            </visual>
+            <!-- Collision cylinder -->
+            <collision>
+                <origin xyz="0 0 0" rpy="0 0 0" />
+                <geometry>
+                    <cylinder length="0.06" radius="${radius}" />
+                </geometry>
+                <material name="Black" />
+            </collision>
+        </link>
+        <joint name="wheel_${type}_joint" type="${mimic_type}">
+            <origin xyz="-0.221 ${orientation * -0.235} -0.05" rpy="${orientation * M_PI/2} 0 0" />
+            <parent link="${parent}" />
+            <child link="wheel_${type}" />
+            <axis xyz="0 0 ${-1 * orientation}" />
+        </joint>
+        <link name="wheel_${type}">
+            <inertial>
+                <mass value="3" />
+                <inertia ixx="1e-3" ixy="0.0" ixz="0.0"
+                    iyy="1e-3" iyz="0.0"
+                    izz="1e-3" />
+            </inertial>
+            <visual>
+                <origin xyz="0 0 0" rpy="0 0 0" />
+                <geometry>
+                    <mesh filename="${path_meshes}/wheel.stl" scale="${scale} ${scale} ${scale}" />
+                    <cylinder length="0.06" radius="${radius_wheel}" />
+                </geometry>
+                <material name="Black" />
+            </visual>
+            <!-- Collision cylinder -->
+            <collision>
+                <origin xyz="0 0 0" rpy="0 0 0" />
+                <geometry>
+                    <cylinder length="0.06" radius="${radius_wheel}" />
                 </geometry>
                 <material name="Black" />
@@ -52,4 +116,19 @@
         </link>
         <gazebo reference="sprocket_${type}">
+            <material>Gazebo/Blue</material>
+            <kp>10000000</kp>
+            <kd>10000000</kd>
+            <mu1>0</mu1>
+            <mu2>0</mu2>
+            <!-- Ignition color reference -->
+            <visual>
+                <material>
+                    <ambient>0.0 0.0 0.5 1.0</ambient>
+                    <diffuse>0.0 0.0 0.5 1.0</diffuse>
+                    <specular>0.0 0.0 0.5 1.0</specular>
+                </material>
+            </visual>
+        </gazebo>
+        <gazebo reference="drive_${type}">
             <material>Gazebo/Blue</material>
             <kp>10000000</kp>
@@ -66,34 +145,4 @@
             </visual>
         </gazebo>
-        <joint name="wheel_${type}_joint" type="${mimic_type}">
-            <origin xyz="-0.442 ${orientation * -0.235} -0.05" rpy="${orientation * M_PI/2} 0 0" />
-            <parent link="${parent}"/>
-            <child link="wheel_${type}"/>
-            <axis xyz="0 0 ${-1 * orientation}" />
-        </joint>
-        <link name="wheel_${type}">
-        <inertial>
-            <mass value="3" />
-            <inertia ixx="1e-3" ixy="0.0" ixz="0.0"
-                 iyy="1e-3" iyz="0.0"
-                 izz="1e-3" />
-        </inertial>
-            <visual>
-                <origin xyz="0 0 0" rpy="0 0 0" />
-                <geometry>
-                    <mesh filename="${path_meshes}/wheel.stl" scale="${scale} ${scale} ${scale}"/>
-                    <cylinder length="0.06" radius="${radius_wheel}"/>
-                </geometry>
-                <material name="Black" />
-            </visual>
-            <!-- Collision cylinder -->
-            <collision>
-                <origin xyz="0 0 0" rpy="0 0 0" />
-                <geometry>
-                    <cylinder length="0.06" radius="${radius_wheel}"/>
-                </geometry>
-                <material name="Black" />
-            </collision>
-        </link>
         <gazebo reference="wheel_${type}">
             <material>Gazebo/Red</material>
@@ -112,7 +161,7 @@
         </gazebo>
         <joint name="track_${type}_joint" type="fixed">
-            <origin xyz="-0.221 ${orientation * -0.235} -0.05" rpy="${orientation * M_PI/2} 0 0" />
-            <parent link="${parent}"/>
-            <child link="track_${type}"/>
+            <origin xyz="0 ${orientation * -0.235} -0.05" rpy="${orientation * M_PI/2} 0 0" />
+            <parent link="${parent}" />
+            <child link="track_${type}" />
         </joint>
         <link name="track_${type}">
@@ -120,5 +169,5 @@
                 <origin xyz="0 0 0" rpy="${M_PI/2} 0 0" />
                 <geometry>
-                    <mesh filename="${path_meshes}/track.stl" scale="${scale} ${scale} ${scale}"/>
+                    <mesh filename="${path_meshes}/track.stl" scale="${scale} ${scale} ${scale}" />
                 </geometry>
                 <material name="Black" />

File: src/tracked_robot_description/urdf/tracked_robot_core.urdf.xacro (robot description, xacro)
@@ -1,3 +1,3 @@
-<?xml version="1.0" ?>
+<?xml version="1.0"?>
 <robot name="tracked_robot" xmlns:xacro="http://ros.org/wiki/xacro">
     <xacro:include filename="track.urdf.xacro" />
@@ -7,49 +7,55 @@
     <xacro:include filename="gps.urdf.xacro" />
     <material name="Black">
-        <color rgba="0.1 0.1 0.1 1.0"/>
+        <color rgba="0.1 0.1 0.1 1.0" />
     </material>
     <material name="Green">
-        <color rgba="0.0 0.8 0.0 1.0"/>
+        <color rgba="0.0 0.8 0.0 1.0" />
     </material>
     <material name="aluminum">
-        <color rgba="0.5 0.5 0.5 1.0"/>
+        <color rgba="0.5 0.5 0.5 1.0" />
     </material>
     <material name="DarkGrey">
-        <color rgba="0.3 0.3 0.3 1.0"/>
+        <color rgba="0.3 0.3 0.3 1.0" />
     </material>
     <material name="GunMetalGrey">
-        <color rgba="0.46 0.5 0.56 1.0"/>
+        <color rgba="0.46 0.5 0.56 1.0" />
     </material>
     <material name="Gold">
         <color rgba="1 1 0.752941176470588 1" />
     </material>
+    <material name="Red">
+        <color rgba="1 0 0 1" />
+    </material>
     <material name="zedm_mat">
-        <color rgba="0 0 0 0.9"/>
+        <color rgba="0 0 0 0.9" />
     </material>
-    <xacro:property name="M_PI" value="3.14159"/>
-    <xacro:property name="sprocket_radius" value="0.069"/>
-    <xacro:macro name="robot" params="diff_drive_emulation mimic_enable:=true path_meshes:=package://tracked_robot_description/meshes">
-<link name="base_footprint"/>
-  <!-- The base footprint of the robot is located underneath the chassis -->
-  <joint name="base_joint" type="fixed">
-    <parent link="base_footprint"/>
-    <child link="base_link" />
-    <origin xyz="0.0 0.0 0.1" rpy="0 0 0"/>
-  </joint>
-    <link name="base_link">
-        <visual>
-            <origin xyz="-0.221 0 -0.05" rpy="1.5707963267949 0 ${M_PI}"/>
-            <geometry>
-                <mesh filename="${path_meshes}/robot_base.stl" scale="1 1 1" />
-            </geometry>
-            <material name="Green" />
-        </visual>
-    </link>
-    <xacro:track type="left" parent="base_link" radius="${sprocket_radius}" diff_drive_emulation="${diff_drive_emulation}" mimic_enable="${mimic_enable}"/>
-    <xacro:track type="right" parent="base_link" radius="${sprocket_radius}" diff_drive_emulation="${diff_drive_emulation}" mimic_enable="${mimic_enable}"/>
-    <xacro:hand parent="base_link" />
-    <xacro:lidar parent="base_link" />
-    <xacro:imu parent="base_link" />
-    <xacro:gps parent="base_link" />
+    <xacro:property name="M_PI" value="3.14159" />
+    <xacro:property name="sprocket_radius" value="0.069" />
+    <xacro:macro name="robot"
+        params="diff_drive_emulation mimic_enable:=true path_meshes:=package://tracked_robot_description/meshes">
+        <link name="base_footprint" />
+        <!-- The base footprint of the robot is located underneath the chassis -->
+        <joint name="base_joint" type="fixed">
+            <parent link="base_footprint" />
+            <child link="base_link" />
+            <origin xyz="0.0 0.0 0.1" rpy="0 0 0" />
+        </joint>
+        <link name="base_link">
+            <visual>
+                <origin xyz="0 0 -0.05" rpy="1.5707963267949 0 ${M_PI}" />
+                <geometry>
+                    <mesh filename="${path_meshes}/robot_base.stl" scale="1 1 1" />
+                </geometry>
+                <material name="Green" />
+            </visual>
+        </link>
+        <xacro:track type="left" parent="base_link" radius="${sprocket_radius}"
+            diff_drive_emulation="${diff_drive_emulation}" mimic_enable="${mimic_enable}" />
+        <xacro:track type="right" parent="base_link" radius="${sprocket_radius}"
+            diff_drive_emulation="${diff_drive_emulation}" mimic_enable="${mimic_enable}" />
+        <xacro:hand parent="base_link" />
+        <xacro:lidar parent="base_link" />
+        <xacro:imu parent="base_link" />
+        <xacro:gps parent="base_link" />
     </xacro:macro>
 </robot>

File: src/tracked_robot_gazebo/urdf/diff_drive.gazebo.xacro (robot description, xacro)
@@ -7,6 +7,9 @@
             <!-- Plugin update rate in Hz -->
             <update_rate>${update_rate}</update_rate>
-            <num_wheel_pairs>2</num_wheel_pairs>
+            <num_wheel_pairs>3</num_wheel_pairs>
             <!-- Name of left joint, defaults to `left_joint` -->
+            <left_joint>drive_left_joint</left_joint>
+            <!-- Name of right joint, defaults to `right_joint` -->
+            <right_joint>drive_right_joint</right_joint>
             <left_joint>sprocket_left_joint</left_joint>
             <!-- Name of right joint, defaults to `right_joint` -->
@@ -43,6 +46,6 @@
             </ros>
             <update_rate>${update_rate}</update_rate>
-            <joint_name>sprocket_left_joint</joint_name>
-            <joint_name>sprocket_right_joint</joint_name>
+            <joint_name>drive_left_joint</joint_name>
+            <joint_name>drive_right_joint</joint_name>
             <joint_name>wheel_left_joint</joint_name>
             <joint_name>wheel_right_joint</joint_name>
