Commit message: Fix robot rotation center

File: src/tracked_robot_gazebo/urdf/gps.gazebo.xacro (robot description, xacro)
@@ -1,23 +1,21 @@
 <?xml version="1.0"?>
 <robot name="tracked_robot" xmlns:xacro="http://ros.org/wiki/xacro">
-    <xacro:macro name="track_gps" params="parent update_rate">
+  <xacro:macro name="track_gps" params="parent update_rate">
     <gazebo reference="gps_link">
-    <sensor name="gps_sensor" type="gps">
-      <!-- ensure the sensor is active (required) -->
-      <always_on>true</always_on>
-      <update_rate>30</update_rate>
-      <plugin name="gps_plugin" filename="libgazebo_ros_gps_sensor.so">
-        <ros>
-          <!-- publish to /gps/fix -->
-          <namespace>/gps</namespace>
-          <remapping>~/out:=fix</remapping>
-          <remapping>~/vel:=velocity</remapping>
-        </ros>
-        <output_type>sensor_msgs/NavSatFix</output_type>
-        <frame_name>gps_link</frame_name>
-      </plugin>
-    </sensor>
-        <material>Gazebo/Grey</material>
+      <sensor name="gps_sensor" type="gps">
+        <always_on>true</always_on>
+        <update_rate>30</update_rate>
+        <plugin name="gps_plugin" filename="libgazebo_ros_gps_sensor.so">
+          <ros>
+            <namespace>/gps</namespace>
+            <remapping>~/out:=fix</remapping>
+            <remapping>~/vel:=velocity</remapping>
+          </ros>
+          <output_type>sensor_msgs/NavSatFix</output_type>
+          <frame_name>gps_link</frame_name>
+        </plugin>
+      </sensor>
+      <material>Gazebo/Grey</material>
     </gazebo>
-    </xacro:macro>
+  </xacro:macro>
 </robot>
