Commit message: Fix transformation, resize model to real size

File: src/tracked_robot_description/urdf/camera.urdf.xacro (robot description, xacro)
@@ -1,28 +1,29 @@
 <?xml version="1.0"?>
 <robot name="tracked_robot" xmlns:xacro="http://ros.org/wiki/xacro">
-    <xacro:macro name="camera"  params="parent">
+    <xacro:macro name="camera" params="parent">
         <joint name="camera_sensor_joint" type="fixed">
-            <origin xyz="0.6 0 -0.015" rpy="0 ${M_PI/2} 0"/>
-            <parent link="${parent}"/>
-            <child link="camera_link"/>
+            <origin xyz="0.27 0 -0.015" rpy="0 ${M_PI/2} 0" />
+            <parent link="${parent}" />
+            <child link="camera_link" />
         </joint>
         <link name="camera_link">
             <collision>
-            <origin xyz="0 0 0" rpy="0 0 0"/>
-            <geometry>
-                <box size="0.1 0.1 0.1"/>
-            </geometry>
+                <origin xyz="0 0 0" rpy="0 0 0" />
+                <geometry>
+                    <box size="0.02 0.02 0.02" />
+                </geometry>
             </collision>
             <visual>
-                <origin xyz="0 0 0" rpy="0 0 0"/>
-            <geometry>
-                <box size="0.02 0.02 0.02"/>
-            </geometry>
-            <material name="Red"/>
+                <origin xyz="0 0 0" rpy="0 0 0" />
+                <geometry>
+                    <box size="0.02 0.02 0.02" />
+                </geometry>
+                <material name="Red" />
             </visual>
             <inertial>
-                <mass value="0.001"/>
-                <origin rpy=" 0 0 0" xyz="0 0 0"/>
-                <inertia ixx="1.6666666666666668e-07" ixy="0" ixz="0" iyy="1.6666666666666668e-07" iyz="0" izz="1.6666666666666668e-07"/>
+                <mass value="0.001" />
+                <origin rpy=" 0 0 0" xyz="0 0 0" />
+                <inertia ixx="1.6666666666666668e-07" ixy="0" ixz="0" iyy="1.6666666666666668e-07"
+                    iyz="0" izz="1.6666666666666668e-07" />
             </inertial>
         </link>

File: src/tracked_robot_description/urdf/hand.urdf.xacro (robot description, xacro)
@@ -2,37 +2,37 @@
 <robot name="tracked_robot" xmlns:xacro="http://ros.org/wiki/xacro">
     <xacro:include filename="camera.urdf.xacro" />
-    <xacro:macro name="hand"  params="parent">
+    <xacro:macro name="hand" params="parent">
         <joint name="hand_base_joint" type="fixed">
-            <origin xyz="-0.180 0 0.14" rpy="0 0 0" />
-            <parent link="${parent}"/>
-            <child link="hand_base"/>
+            <origin xyz="0.0 0 0.09" rpy="0 0 0" />
+            <parent link="${parent}" />
+            <child link="hand_base" />
             <axis xyz="0 0 1" />
         </joint>
         <link name="hand_base">
-        <inertial>
-            <mass value="2" />
-            <inertia ixx="1e-3" ixy="0.0" ixz="0.0"
-                 iyy="1e-3" iyz="0.0"
-                 izz="1e-3" />
-        </inertial>
+            <inertial>
+                <mass value="0.2" />
+                <inertia ixx="1e-3" ixy="0.0" ixz="0.0"
+                    iyy="1e-3" iyz="0.0"
+                    izz="1e-3" />
+            </inertial>
             <visual>
-                <origin xyz="0 0 0" rpy="0 0 0"/>
+                <origin xyz="0 0 0" rpy="0 0 0" />
                 <geometry>
-                     <cylinder length="0.18" radius="0.06"/>
+                    <cylinder length="0.04" radius="0.02" />
                 </geometry>
                 <material name="Black" />
             </visual>
         </link>
-       <joint name="hand_joint" type="fixed">
-            <origin xyz="0 0 0.09" rpy="0 0 0" />
-            <parent link="hand_base"/>
-            <child link="hand"/>
+        <joint name="hand_joint" type="fixed">
+            <origin xyz="0 0 0.02" rpy="0 0 0" />
+            <parent link="hand_base" />
+            <child link="hand" />
             <axis xyz="0 0 1" />
         </joint>
         <link name="hand">
             <visual>
-                <origin xyz="0.3 0 0" rpy="0 0 0"/>
+                <origin xyz="0.135 0 0" rpy="0 0 0" />
                 <geometry>
-                     <box size="0.7 0.1 0.01"/>
+                    <box size="0.3 0.03 0.01" />
                 </geometry>
                 <material name="Black" />

File: src/tracked_robot_description/urdf/imu.urdf.xacro (robot description, xacro)
@@ -1,28 +1,29 @@
 <?xml version="1.0"?>
 <robot name="tracked_robot" xmlns:xacro="http://ros.org/wiki/xacro">
-    <xacro:macro name="imu"  params="parent">
+    <xacro:macro name="imu" params="parent">
         <joint name="imu_sensor_joint" type="fixed">
-            <origin xyz="0 0 0" rpy="0 0 0"/>
-            <parent link="${parent}"/>
-            <child link="imu_link"/>
+            <origin xyz="0 0 0" rpy="0 0 0" />
+            <parent link="${parent}" />
+            <child link="imu_link" />
         </joint>
         <link name="imu_link">
             <collision>
-            <origin xyz="0 0 0" rpy="0 0 0"/>
-            <geometry>
-            <box size="0.1 0.1 0.1"/>
-            </geometry>
+                <origin xyz="0 0 0" rpy="0 0 0" />
+                <geometry>
+                    <box size="0.02 0.02 0.02" />
+                </geometry>
             </collision>
             <visual>
-            <origin xyz="0 0 0" rpy="0 0 0"/>
-            <geometry>
-                <box size="0.02 0.02 0.02"/>
-            </geometry>
-            <material name="Red"/>
+                <origin xyz="0 0 0" rpy="0 0 0" />
+                <geometry>
+                    <box size="0.02 0.02 0.02" />
+                </geometry>
+                <material name="Red" />
             </visual>
             <inertial>
-                <mass value="0.001"/>
-                <origin rpy=" 0 0 0" xyz="0 0 0"/>
-                <inertia ixx="1.6666666666666668e-07" ixy="0" ixz="0" iyy="1.6666666666666668e-07" iyz="0" izz="1.6666666666666668e-07"/>
+                <mass value="0.001" />
+                <origin rpy=" 0 0 0" xyz="0 0 0" />
+                <inertia ixx="1.6666666666666668e-07" ixy="0" ixz="0" iyy="1.6666666666666668e-07"
+                    iyz="0" izz="1.6666666666666668e-07" />
             </inertial>
         </link>

File: src/tracked_robot_description/urdf/lidar.urdf.xacro (robot description, xacro)
@@ -1,28 +1,34 @@
 <?xml version="1.0"?>
 <robot name="tracked_robot" xmlns:xacro="http://ros.org/wiki/xacro">
-    <xacro:macro name="lidar"  params="parent">
+    <xacro:macro name="lidar" params="parent">
         <joint name="lidar_sensor_joint" type="fixed">
-            <origin xyz="0.0 0 0.11" rpy="0 0 0" />
+            <origin xyz="0.090 0 0.08" rpy="0 0 0" />
+            <parent link="${parent}" />
+            <child link="lidar_link" />
+        </joint>
+        <!-- <joint name="lidar_sensor_joint" type="fixed">
+            <origin xyz="0.0 0 0.11" rpy="0 0 3.141" />
             <parent link="${parent}"/>
             <child link="lidar_link"/>
-        </joint>
+        </joint> -->
         <link name="lidar_link">
             <collision>
-            <origin xyz="0 0 0" rpy="0 0 0"/>
-            <geometry>
-                <cylinder radius="0.05" length="0.04"/>
-            </geometry>
+                <origin xyz="0 0 0" rpy="0 0 0" />
+                <geometry>
+                    <cylinder radius="0.02" length="0.01" />
+                </geometry>
             </collision>
             <visual>
-            <origin xyz="0 0 0" rpy="0 0 0"/>
-            <geometry>
-                <cylinder radius="0.05" length="0.04"/>
-            </geometry>
-            <material name="red"/>
+                <origin xyz="0 0 0" rpy="0 0 0" />
+                <geometry>
+                    <cylinder radius="0.02" length="0.01" />
+                </geometry>
+                <material name="red" />
             </visual>
             <inertial>
-                <mass value="0.001"/>
-                <origin rpy=" 0 0 0" xyz="0 0 0"/>
-                <inertia ixx="1.6666666666666668e-07" ixy="0" ixz="0" iyy="1.6666666666666668e-07" iyz="0" izz="1.6666666666666668e-07"/>
+                <mass value="0.001" />
+                <origin rpy=" 0 0 0" xyz="0 0 0" />
+                <inertia ixx="1.6666666666666668e-07" ixy="0" ixz="0" iyy="1.6666666666666668e-07"
+                    iyz="0" izz="1.6666666666666668e-07" />
             </inertial>
         </link>

File: src/tracked_robot_description/urdf/track.urdf.xacro (robot description, xacro)
@@ -4,39 +4,35 @@
         <!-- Define orientation -->
         <xacro:if value="${type == 'left'}">
-            <xacro:property name="orientation" value="-1"/>
+            <xacro:property name="orientation" value="-1" />
         </xacro:if>
         <xacro:if value="${type == 'right'}">
-            <xacro:property name="orientation" value="1"/>
+            <xacro:property name="orientation" value="1" />
         </xacro:if>
         <xacro:if value="${mimic_enable}">
-            <xacro:property name="mimic_type" value="continuous"/>
+            <xacro:property name="mimic_type" value="continuous" />
         </xacro:if>
         <xacro:unless value="${mimic_enable}">
-            <xacro:property name="mimic_type" value="fixed"/>
+            <xacro:property name="mimic_type" value="fixed" />
         </xacro:unless>
-        <xacro:property name="radius_wheel" value="${radius}"/>
-        <xacro:property name="scale" value="0.0046"/>
+        <xacro:property name="radius_wheel" value="${radius}" />
+        <xacro:property name="scale" value="0.0020" />
         <joint name="sprocket_${type}_joint" type="continuous">
-            <origin xyz="0.0 ${orientation * -0.235} -0.05" rpy="${orientation * M_PI/2} 0 0" />
-            <parent link="${parent}"/>
-            <child link="sprocket_${type}"/>
-            <axis xyz="0 0 ${-1 * orientation}" />
-            <!-- Passive wheel rotate automatically according to the status of the active one -->
-            <xacro:if value="${mimic_enable}">
-                <mimic joint="wheel_${type}_joint" multiplier="1" offset="0"/>
-            </xacro:if>
+            <origin xyz="0.0 ${orientation * -0.106} 0" rpy="0 0 0" />
+            <parent link="${parent}" />
+            <child link="sprocket_${type}" />
+            <axis xyz="0 1 0" />
         </joint>
         <link name="sprocket_${type}">
-         <inertial>
-            <mass value="3" />
-            <inertia ixx="1e-3" ixy="0.0" ixz="0.0"
-                 iyy="1e-3" iyz="0.0"
-                 izz="1e-3" />
-        </inertial>
+            <inertial>
+                <mass value="0.2" />
+                <inertia ixx="1e-3" ixy="0.0" ixz="0.0"
+                    iyy="1e-3" iyz="0.0"
+                    izz="1e-3" />
+            </inertial>
             <visual>
-                <origin xyz="0 0 0" rpy="0 0 0" />
+                <origin xyz="0 0 0" rpy="${pi/2} 0 0" />
                 <geometry>
-                    <mesh filename="${path_meshes}/sprocket.stl" scale="${scale} ${scale} ${scale}"/>
-                    <cylinder length="0.06" radius="${radius_wheel}"/>
+                    <mesh filename="${path_meshes}/sprocket.stl" scale="${scale} ${scale} ${scale}" />
+                    <!-- <cylinder length="0.06" radius="${radius_wheel}" /> -->
                 </geometry>
                 <material name="Black" />
@@ -44,7 +40,7 @@
             <!-- Collision cylinder -->
             <collision>
-                <origin xyz="0 0 0" rpy="0 0 0" />
+                <origin xyz="0 0 0" rpy="${pi/2} 0 0" />
                 <geometry>
-                    <cylinder length="0.06" radius="${radius}"/>
+                    <cylinder length="0.03" radius="0.03" />
                 </geometry>
                 <material name="Black" />
@@ -53,8 +49,8 @@
         <gazebo reference="sprocket_${type}">
             <material>Gazebo/Blue</material>
-            <kp>10000000</kp>
-            <kd>10000000</kd>
-            <mu1>10000000</mu1>
-            <mu2>10000000</mu2>
+            <kp>1e15</kp>
+            <kd>1e13</kd>
+            <mu1>100000</mu1>
+            <mu2>100000</mu2>
             <!-- Ignition color reference -->
             <visual>
@@ -66,22 +62,23 @@
             </visual>
         </gazebo>
-        <joint name="wheel_${type}_joint" type="${mimic_type}">
-            <origin xyz="-0.442 ${orientation * -0.235} -0.05" rpy="${orientation * M_PI/2} 0 0" />
-            <parent link="${parent}"/>
-            <child link="wheel_${type}"/>
-            <axis xyz="0 0 ${-1 * orientation}" />
+        <joint name="wheel_${type}_joint" type="continuous">
+            <origin xyz="-0.092 ${orientation * -0.106} 0" rpy="0 0 0" />
+            <parent link="${parent}" />
+            <child link="wheel_${type}" />
+            <axis xyz="0 1 0" />
+            <mimic joint="sprocket_${type}_joint" multiplier="1" offset="0" />
         </joint>
         <link name="wheel_${type}">
-        <inertial>
-            <mass value="3" />
-            <inertia ixx="1e-3" ixy="0.0" ixz="0.0"
-                 iyy="1e-3" iyz="0.0"
-                 izz="1e-3" />
-        </inertial>
+            <inertial>
+                <mass value="0.2" />
+                <inertia ixx="1e-3" ixy="0.0" ixz="0.0"
+                    iyy="1e-3" iyz="0.0"
+                    izz="1e-3" />
+            </inertial>
             <visual>
-                <origin xyz="0 0 0" rpy="0 0 0" />
+                <origin xyz="0 0 0" rpy="${pi/2} 0 0" />
                 <geometry>
-                    <mesh filename="${path_meshes}/wheel.stl" scale="${scale} ${scale} ${scale}"/>
-                    <cylinder length="0.06" radius="${radius_wheel}"/>
+                    <mesh filename="${path_meshes}/wheel.stl" scale="${scale} ${scale} ${scale}" />
+                    <!-- <cylinder length="0.06" radius="${radius_wheel}" /> -->
                 </geometry>
                 <material name="Black" />
@@ -89,7 +86,7 @@
             <!-- Collision cylinder -->
             <collision>
-                <origin xyz="0 0 0" rpy="0 0 0" />
+                <origin xyz="0 0 0" rpy="${pi/2} 0 0" />
                 <geometry>
-                    <cylinder length="0.06" radius="${radius_wheel}"/>
+                    <cylinder length="0.03" radius="0.03" />
                 </geometry>
                 <material name="Black" />
@@ -98,8 +95,55 @@
         <gazebo reference="wheel_${type}">
             <material>Gazebo/Red</material>
-            <kp>10000000</kp>
-            <kd>10000000</kd>
-            <mu1>0</mu1>
-            <mu2>0</mu2>
+            <kp>1e15</kp>
+            <kd>1e13</kd>
+            <mu1>1</mu1>
+            <mu2>1</mu2>
+            <!-- Ignition color reference -->
+            <visual>
+                <material>
+                    <ambient>0.5 0.0 0.0 1.0</ambient>
+                    <diffuse>0.5 0.0 0.0 1.0</diffuse>
+                    <specular>0.5 0.0 0.0 1.0</specular>
+                </material>
+            </visual>
+        </gazebo>
+        <joint name="front_wheel_${type}_joint" type="continuous">
+            <origin xyz="0.090 ${orientation * -0.106} 0" rpy="0 0 0" />
+            <parent link="${parent}" />
+            <child link="front_wheel_${type}" />
+            <axis xyz="0 1 0" />
+            <!-- Passive wheel rotate automatically according to the status of the active one -->
+            <mimic joint="sprocket_${type}_joint" multiplier="1" offset="0" />
+        </joint>
+        <link name="front_wheel_${type}">
+            <inertial>
+                <mass value="0.2" />
+                <inertia ixx="1e-3" ixy="0.0" ixz="0.0"
+                    iyy="1e-3" iyz="0.0"
+                    izz="1e-3" />
+            </inertial>
+            <visual>
+                <origin xyz="0 0 0" rpy="${pi/2} 0 0" />
+                <geometry>
+                    <mesh filename="${path_meshes}/wheel.stl" scale="${scale} ${scale} ${scale}" />
+                    <!-- <cylinder length="0.06" radius="${radius_wheel}" /> -->
+                </geometry>
+                <material name="Black" />
+            </visual>
+            <!-- Collision cylinder -->
+            <collision>
+                <origin xyz="0 0 0" rpy="${pi/2} 0 0" />
+                <geometry>
+                    <cylinder length="0.03" radius="0.03" />
+                </geometry>
+                <material name="Black" />
+            </collision>
+        </link>
+        <gazebo reference="front_wheel_${type}">
+            <material>Gazebo/Red</material>
+            <kp>1e15</kp>
+            <kd>1e13</kd>
+            <mu1>1</mu1>
+            <mu2>1</mu2>
             <!-- Ignition color reference -->
             <visual>
@@ -112,20 +156,36 @@
         </gazebo>
         <joint name="track_${type}_joint" type="fixed">
-            <origin xyz="-0.221 ${orientation * -0.235} -0.05" rpy="${orientation * M_PI/2} 0 0" />
-            <parent link="${parent}"/>
-            <child link="track_${type}"/>
+            <origin xyz="0.0 ${orientation * -0.106} 0" rpy="0 0 0" />
+            <parent link="${parent}" />
+            <child link="track_${type}" />
         </joint>
         <link name="track_${type}">
+            <inertial>
+                <mass value="0.4" />
+                <inertia ixx="1e-3" ixy="0.0" ixz="0.0"
+                    iyy="1e-3" iyz="0.0"
+                    izz="1e-3" />
+            </inertial>
             <visual>
-                <origin xyz="0 0 0" rpy="${M_PI/2} 0 0" />
+                <origin xyz="0 0 0" rpy="0 0 0" />
                 <geometry>
-                    <mesh filename="${path_meshes}/track.stl" scale="${scale} ${scale} ${scale}"/>
+                    <mesh filename="${path_meshes}/track.stl" scale="${scale} ${scale} ${scale}" />
                 </geometry>
                 <material name="Black" />
             </visual>
+            <collision>
+                <origin xyz="0 0 0" rpy="0 0 0" />
+                <geometry>
+                    <box size="0.225 0.03 0.051" />
+                </geometry>
+                <material name="Black" />
+            </collision>
         </link>
         <gazebo reference="track_${type}">
             <material>Gazebo/Black</material>
-            <!-- Ignition color reference -->
+            <kp>1e15</kp>
+            <kd>1e13</kd>
+            <mu1>0</mu1>
+            <mu2>0</mu2>
             <visual>
                 <material>

File: src/tracked_robot_description/urdf/tracked_robot_core.urdf.xacro (robot description, xacro)
@@ -1,3 +1,3 @@
-<?xml version="1.0" ?>
+<?xml version="1.0"?>
 <robot name="tracked_robot" xmlns:xacro="http://ros.org/wiki/xacro">
     <xacro:include filename="track.urdf.xacro" />
@@ -6,17 +6,17 @@
     <xacro:include filename="imu.urdf.xacro" />
     <material name="Black">
-        <color rgba="0.1 0.1 0.1 1.0"/>
+        <color rgba="0.1 0.1 0.1 1.0" />
     </material>
     <material name="Green">
-        <color rgba="0.0 0.8 0.0 1.0"/>
+        <color rgba="0.0 0.8 0.0 1.0" />
     </material>
     <material name="aluminum">
-        <color rgba="0.5 0.5 0.5 1.0"/>
+        <color rgba="0.5 0.5 0.5 1.0" />
     </material>
     <material name="DarkGrey">
-        <color rgba="0.3 0.3 0.3 1.0"/>
+        <color rgba="0.3 0.3 0.3 1.0" />
     </material>
     <material name="GunMetalGrey">
-        <color rgba="0.46 0.5 0.56 1.0"/>
+        <color rgba="0.46 0.5 0.56 1.0" />
     </material>
     <material name="Gold">
@@ -24,30 +24,46 @@
     </material>
     <material name="zedm_mat">
-        <color rgba="0 0 0 0.9"/>
+        <color rgba="0 0 0 0.9" />
     </material>
-    <xacro:property name="M_PI" value="3.14159"/>
-    <xacro:property name="sprocket_radius" value="0.069"/>
-    <xacro:macro name="robot" params="diff_drive_emulation mimic_enable:=true path_meshes:=package://tracked_robot_description/meshes">
-<link name="base_footprint"/>
-  <!-- The base footprint of the robot is located underneath the chassis -->
-  <joint name="base_joint" type="fixed">
-    <parent link="base_footprint"/>
-    <child link="base_link" />
-    <origin xyz="0.0 0.0 0.1" rpy="0 0 0"/>
-  </joint>
-    <link name="base_link">
-        <visual>
-            <origin xyz="-0.221 0 -0.05" rpy="1.5707963267949 0 ${M_PI}"/>
-            <geometry>
-                <mesh filename="${path_meshes}/robot_base.stl" scale="1 1 1" />
-            </geometry>
-            <material name="Green" />
-        </visual>
-    </link>
-    <xacro:track type="left" parent="base_link" radius="${sprocket_radius}" diff_drive_emulation="${diff_drive_emulation}" mimic_enable="${mimic_enable}"/>
-    <xacro:track type="right" parent="base_link" radius="${sprocket_radius}" diff_drive_emulation="${diff_drive_emulation}" mimic_enable="${mimic_enable}"/>
-    <xacro:hand parent="base_link" />
-    <xacro:lidar parent="base_link" />
-    <xacro:imu parent="base_link" />
+    <xacro:property name="M_PI" value="3.14159" />
+    <xacro:property name="sprocket_radius" value="0.059" />
+    <xacro:macro name="robot"
+        params="diff_drive_emulation mimic_enable:=true path_meshes:=package://tracked_robot_description/meshes">
+        <link name="base_footprint" />
+        <!-- The base footprint of the robot is located underneath the chassis -->
+        <joint name="base_joint" type="fixed">
+            <parent link="base_footprint" />
+            <child link="base_link" />
+            <origin xyz="0.0 0.0 0.0" rpy="0 0 0" />
+        </joint>
+        <link name="base_link">
+            <inertial>
+                <mass value="1.0" />
+                <inertia ixx="1e-3" ixy="0.0" ixz="0.0"
+                    iyy="1e-3" iyz="0.0"
+                    izz="1e-3" />
+            </inertial>
+            <visual>
+                <origin xyz="0.0 0 0" rpy="1.5707963267949 0 ${M_PI}" />
+                <geometry>
+                    <mesh filename="${path_meshes}/robot_base.stl" scale="0.363 0.507 0.450" />
+                </geometry>
+                <material name="Green" />
+            </visual>
+            <collision>
+                <origin xyz="0 0 0.00" rpy="0 0 0" />
+                <geometry>
+                    <box size="0.231 0.196 0.051" />
+                </geometry>
+                <material name="Black" />
+            </collision>
+        </link>
+        <xacro:track type="left" parent="base_link" radius="${sprocket_radius}"
+            diff_drive_emulation="${diff_drive_emulation}" mimic_enable="${mimic_enable}" />
+        <xacro:track type="right" parent="base_link" radius="${sprocket_radius}"
+            diff_drive_emulation="${diff_drive_emulation}" mimic_enable="${mimic_enable}" />
+        <xacro:lidar parent="base_link" />
+        <xacro:hand parent="base_link" />
+        <xacro:imu parent="base_link" />
     </xacro:macro>
 </robot>
