Commit message: Fix transformation, resize model to real size

File: src/tracked_robot_gazebo/urdf/diff_drive.gazebo.xacro (robot description, xacro)
@@ -1,51 +1,34 @@
 <?xml version="1.0"?>
 <robot name="tracked_robot" xmlns:xacro="http://ros.org/wiki/xacro">
-    <!--Reference http://gazebosim.org/tutorials?tut=ros_gzplugins#DifferentialDrive -->
-    <xacro:macro name="track_drive" params="parent robot_name update_rate wheel_radius wheel_separation publish_odom_tf">
+    <!--Reference
+    http://gazebosim.org/tutorials?tut=ros_gzplugins#DifferentialDrive -->
+    <xacro:macro name="track_drive"
+        params="parent robot_name update_rate wheel_radius wheel_separation publish_odom_tf">
+        <ros2_control name="GazeboSystem" type="system">
+            <hardware>
+                <plugin>gazebo_ros2_control/GazeboSystem</plugin>
+            </hardware>
+            <joint name="sprocket_left_joint">
+                <command_interface name="velocity">
+                </command_interface>
+                <state_interface name="position" />
+                <state_interface name="velocity" />
+            </joint>
+            <joint name="sprocket_right_joint">
+                <command_interface name="velocity">
+                </command_interface>
+                <state_interface name="position" />
+                <state_interface name="velocity" />
+            </joint>
+        </ros2_control>
         <gazebo>
-            <plugin filename="libgazebo_ros_diff_drive.so" name="skid_steer_drive_controller">
-            <!-- Plugin update rate in Hz -->
-            <update_rate>${update_rate}</update_rate>
-            <num_wheel_pairs>2</num_wheel_pairs>
-            <!-- Name of left joint, defaults to `left_joint` -->
-            <left_joint>sprocket_left_joint</left_joint>
-            <!-- Name of right joint, defaults to `right_joint` -->
-            <right_joint>sprocket_right_joint</right_joint>
-            <left_joint>wheel_left_joint</left_joint>
-            <!-- Name of right joint, defaults to `right_joint` -->
-            <right_joint>wheel_right_joint</right_joint>
-            <!-- The distance from the center of one wheel to the other, in meters, defaults to 0.34 m -->
-            <wheel_separation>${wheel_separation}</wheel_separation>
-            <!-- Diameter of the wheels, in meters, defaults to 0.15 m -->
-            <wheel_diameter>${wheel_radius * 2}</wheel_diameter>
-            <!-- Wheel acceleration, in rad/s^2, defaults to 0.0 rad/s^2 -->
-            <wheel_acceleration>0.2</wheel_acceleration>
-            <!-- Maximum torque which the wheels can produce, in Nm, defaults to 5 Nm -->
-            <max_wheel_torque>5</max_wheel_torque>
-            <!-- Odometry frame, defaults to `odom` -->
-            <odometry_frame>odom</odometry_frame>
-            <!-- Robot frame to calculate odometry from, defaults to `base_footprint` -->
-            <robot_base_frame>${parent}</robot_base_frame>
-            <!-- Set to true to publish transforms for the odometry, defaults to true -->
-            <publish_odom>true</publish_odom>
-            <publish_odom_tf>${publish_odom_tf}</publish_odom_tf>
-            <!-- Set to true to publish transforms for the wheel links, defaults to false -->
-            <publish_wheel_tf>false</publish_wheel_tf>
-            <!-- Odometry source, 0 for ENCODER, 1 for WORLD, defaults to WORLD -->
-            <odometry_source>1</odometry_source>
-            <!-- Set to true to publish sensor_msgs/JointState on /joint_states for the wheel joints, defaults to false -->
-            <publis_wheel_joint_state>false</publis_wheel_joint_state>
+            <!-- Joint state publisher -->
+            <plugin filename="libgazebo_ros2_control.so" name="gazebo_ros2_control">
+                <parameters>$(find tracked_robot_hardware)/controllers/robot_controller.yaml</parameters>
+                <ros>
+                    <remapping>diff_drive_base_controller/cmd_vel_unstamped:=cmd_vel</remapping>
+                    <remapping>diff_drive_base_controller/odom:=odom</remapping>
+                </ros>
             </plugin>
-            <plugin name="basic_mobile_bot_joint_state"
-            filename="libgazebo_ros_joint_state_publisher.so">
-            <ros>
-                <remapping>~/out:=joint_states</remapping>
-            </ros>
-            <update_rate>${update_rate}</update_rate>
-            <joint_name>sprocket_left_joint</joint_name>
-            <joint_name>sprocket_right_joint</joint_name>
-            <joint_name>wheel_left_joint</joint_name>
-            <joint_name>wheel_right_joint</joint_name>
-        </plugin>
         </gazebo>
     </xacro:macro>

File: src/tracked_robot_gazebo/urdf/imu.gazebo.xacro (robot description, xacro)
@@ -1,72 +1,72 @@
 <?xml version="1.0"?>
 <robot name="tracked_robot" xmlns:xacro="http://ros.org/wiki/xacro">
-    <xacro:macro name="track_imu" params="parent">
-   <gazebo reference="imu_link">
-    <sensor name="imu_sensor" type="imu">
-      <plugin filename="libgazebo_ros_imu_sensor.so" name="imu_plugin">
-        <ros>
-          <namespace>/imu</namespace>
-          <remapping>~/out:=data</remapping>
-        </ros>
-         <always_on>true</always_on>
-      <update_rate>100</update_rate>
-      <visualize>true</visualize>
-      <imu>
-        <angular_velocity>
-          <x>
-            <noise type="gaussian">
-              <mean>0.0</mean>
-              <stddev>2e-4</stddev>
-              <bias_mean>0.0000075</bias_mean>
-              <bias_stddev>0.0000008</bias_stddev>
-            </noise>
-          </x>
-          <y>
-            <noise type="gaussian">
-              <mean>0.0</mean>
-              <stddev>2e-4</stddev>
-              <bias_mean>0.0000075</bias_mean>
-              <bias_stddev>0.0000008</bias_stddev>
-            </noise>
-          </y>
-          <z>
-            <noise type="gaussian">
-              <mean>0.0</mean>
-              <stddev>2e-4</stddev>
-              <bias_mean>0.0000075</bias_mean>
-              <bias_stddev>0.0000008</bias_stddev>
-            </noise>
-          </z>
-        </angular_velocity>
-        <linear_acceleration>
-          <x>
-            <noise type="gaussian">
-              <mean>0.0</mean>
-              <stddev>1.7e-2</stddev>
-              <bias_mean>0.1</bias_mean>
-              <bias_stddev>0.001</bias_stddev>
-            </noise>
-          </x>
-          <y>
-            <noise type="gaussian">
-              <mean>0.0</mean>
-              <stddev>1.7e-2</stddev>
-              <bias_mean>0.1</bias_mean>
-              <bias_stddev>0.001</bias_stddev>
-            </noise>
-          </y>
-          <z>
-            <noise type="gaussian">
-              <mean>0.0</mean>
-              <stddev>1.7e-2</stddev>
-              <bias_mean>0.1</bias_mean>
-              <bias_stddev>0.001</bias_stddev>
-            </noise>
-          </z>
-        </linear_acceleration>
-      </imu>
-      </plugin>
-    </sensor>
-  </gazebo>
-    </xacro:macro>
+  <xacro:macro name="track_imu" params="parent">
+    <gazebo reference="imu_link">
+      <sensor name="imu_sensor" type="imu">
+        <plugin filename="libgazebo_ros_imu_sensor.so" name="imu_plugin">
+          <ros>
+            <namespace>/imu</namespace>
+            <remapping>~/out:=data</remapping>
+          </ros>
+          <always_on>true</always_on>
+          <update_rate>100</update_rate>
+          <visualize>true</visualize>
+          <imu>
+            <angular_velocity>
+              <x>
+                <noise type="gaussian">
+                  <mean>0.0</mean>
+                  <stddev>2e-4</stddev>
+                  <bias_mean>0.0000075</bias_mean>
+                  <bias_stddev>0.0000008</bias_stddev>
+                </noise>
+              </x>
+              <y>
+                <noise type="gaussian">
+                  <mean>0.0</mean>
+                  <stddev>2e-4</stddev>
+                  <bias_mean>0.0000075</bias_mean>
+                  <bias_stddev>0.0000008</bias_stddev>
+                </noise>
+              </y>
+              <z>
+                <noise type="gaussian">
+                  <mean>0.0</mean>
+                  <stddev>2e-4</stddev>
+                  <bias_mean>0.0000075</bias_mean>
+                  <bias_stddev>0.0000008</bias_stddev>
+                </noise>
+              </z>
+            </angular_velocity>
+            <linear_acceleration>
+              <x>
+                <noise type="gaussian">
+                  <mean>0.0</mean>
+                  <stddev>1.7e-2</stddev>
+                  <bias_mean>0.1</bias_mean>
+                  <bias_stddev>0.001</bias_stddev>
+                </noise>
+              </x>
+              <y>
+                <noise type="gaussian">
+                  <mean>0.0</mean>
+                  <stddev>1.7e-2</stddev>
+                  <bias_mean>0.1</bias_mean>
+                  <bias_stddev>0.001</bias_stddev>
+                </noise>
+              </y>
+              <z>
+                <noise type="gaussian">
+                  <mean>0.0</mean>
+                  <stddev>1.7e-2</stddev>
+                  <bias_mean>0.1</bias_mean>
+                  <bias_stddev>0.001</bias_stddev>
+                </noise>
+              </z>
+            </linear_acceleration>
+          </imu>
+        </plugin>
+      </sensor>
+    </gazebo>
+  </xacro:macro>
 </robot>
